File: tito/Placa_Tito_2013/Placa_principal/placa_principal.kicad_pcb (KiCad board)
At the start: 2 copper layers, 65 x 100 mm, 76 parts, among them IC1 ATMEGA88-P, K1 Servo, K2 Jumper con doble posicion, P1 Puerto Serie, P2 Motor 1, P3 Motor 2, P4 Bateria 3,6V, P5 Bateria 7,2V, P6 Programador, P7 CONN_1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

Commit message: Mas ruteo, incompleto
Parts:
- R1, R10, R11, R12, R13, R2, R4, R5, R6, R7, R8, R9: footprint R3 -> R1
- moved JP1 194.3 mm to (50.0, 63.0)
- moved R10 140.2 mm to (47.0, 83.0), turned to 0 degrees
- moved C7 139.6 mm to (46.0, 65.0), turned to 270 degrees
- moved D10 130.8 mm to (112.0, 160.0)
- moved D11 130.8 mm to (112.0, 154.0)
- moved D12 130.8 mm to (112.0, 157.0)
- moved D9 130.8 mm to (112.0, 163.0)
- moved JP2 130.8 mm to (130.0, 160.0)
- moved R15 130.8 mm to (120.0, 163.0)
- moved R16 130.8 mm to (120.0, 160.0)
- moved R17 130.8 mm to (120.0, 154.0)
- moved R18 130.8 mm to (120.0, 157.0)
- moved P6 126.0 mm to (242.0, 152.0), turned to 270 degrees
- moved R14 125.9 mm to (184.0, 150.0), turned to 90 degrees
- moved R12 125.3 mm to (55.0, 83.0), turned to 0 degrees
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
Commit message: Se terminaron de acomodar los componentes en la placa, y se inició el routeo de la misma
Parts:
- removed the 1PIN at (87.0, 152.0) (x2)
- removed the 1PIN at (32.0, 152.0)
- removed the 1PIN at (32.0, 135.0)
- removed the 1PIN at (87.0, 135.0)
- added 1PIN2mm: P***, 1PIN2mm, F.Cu at (32.0, 135.0)
- added 1PIN2mm: P***, 1PIN2mm, F.Cu at (32.0, 152.0)
- added 1PIN2mm: P***, 1PIN2mm, F.Cu at (87.0, 152.0)
- added 1PIN2mm: P***, 1PIN2mm, F.Cu at (87.0, 135.0)
- added 1PIN2mm: P***, 1PIN2mm, F.Cu at (59.5, 65.0)
- added JP3: JUMPER, PIN_ARRAY_2X1, F.Cu at (69.0, 108.0)
- C5: footprint C1 -> SM0805; moved to B.Cu
- P7, P8, P9: footprint 1pin -> 1PIN2mm
- U8: moved to B.Cu
- moved SW3 238.9 mm to (35.5, 107.5), turned to 270 degrees
- moved R19 232.3 mm to (45.0, 105.5), turned to 180 degrees
- moved P9 231.5 mm to (38.0, 101.0)
- moved P4 194.6 mm to (87.0, 96.5), turned to 90 degrees
- moved D8 194.0 mm to (78.0, 88.5)
- moved D4 194.0 mm to (78.0, 98.0)
- moved D7 191.5 mm to (75.5, 88.5)
- moved D3 191.5 mm to (75.5, 98.0)
- moved P3 190.5 mm to (72.5, 93.5)
- moved U5 189.5 mm to (59.5, 93.5)
- moved P2 188.5 mm to (46.5, 93.5)
- moved C2 187.6 mm to (56.5, 86.0), turned to 0 degrees
- moved D5 186.5 mm to (43.5, 88.5)
- moved D1 186.5 mm to (43.5, 98.0)
- moved U8 184.1 mm to (78.9, 135.5)
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Connections:
- R3 pad 2: /SCK -> N-0000047
- SW1 pad 1: /SCK -> N-0000047
Routing:
- net GND: track 0.00 -> 116.4 mm
- net /MOSI: track 0.00 -> 69.9 mm, vias 0 -> 3
- net /RESET: track 0.00 -> 67.0 mm
- net +5V: track 0.00 -> 48.0 mm
- net N-0000047: track 0.00 -> 28.2 mm
- net /SCK: track 0.00 -> 23.9 mm
- net /LED2: track 0.00 -> 21.3 mm
- net N-0000056: track 0.00 -> 19.3 mm
- net N-0000021: track 0.00 -> 13.7 mm
- net /TX: track 0.00 -> 11.2 mm
- net /RX: track 0.00 -> 11.2 mm
- net +8V: track 0.00 -> 6.51 mm
- net N-0000014: track 0.00 -> 4.83 mm
- net N-0000015: track 0.00 -> 4.74 mm
- net N-0000019: track 0.00 -> 3.19 mm
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Other:
- net class Default: clearance 0.254 -> 0.3048; trace_width 1.00076 -> 0.3048
- net class TrueHole: clearance 0.254 -> 0.3048
- rule trace_clearance: 0.254 -> 0.3048

Commit message: Casi finalizamos de routear la placa
Parts:
- R1, R10, R11, R12, R13, R2, R4, R5, R6, R7: footprint R1 -> R3
- R15, R16, R17, R18: footprint R3 -> SM0805
- moved K1 23.3 mm to (90.0, 68.6), turned to 270 degrees
- moved R12 13.9 mm to (48.6, 63.7), turned to 90 degrees
- moved R7 13.9 mm to (76.8, 77.6)
- moved R6 12.9 mm to (84.7, 64.8)
- moved R4 12.6 mm to (32.8, 76.0), turned to 90 degrees
- moved R11 12.4 mm to (77.5, 64.9)
- moved RV4 12.3 mm to (81.0, 77.0)
- moved RV2 11.8 mm to (35.8, 64.2)
- moved RV1 11.6 mm to (35.8, 76.0)
- moved RV3 11.4 mm to (80.5, 65.1)
- moved R13 11.3 mm to (84.0, 75.0)
- moved R5 10.8 mm to (32.8, 64.2)
- moved JP2 7.50 mm to (62.0, 131.3), turned to 0 degrees
- moved R10 3.63 mm to (41.0, 67.1), turned to 90 degrees
Connections:
- IC1 pad 13: /LED4 -> /LED3
- IC1 pad 18: /LED2 -> /LED4
- IC1 pad 23: /SENSOR 1 -> /SENSOR 4
- IC1 pad 24: /SENSOR 2 -> /SENSOR 3
- IC1 pad 25: /SENSOR 3 -> /SENSOR 2
- IC1 pad 26: /SENSOR 4 -> /SENSOR 1
- IC1 pad 6: /LED3 -> /LED2
- JP2 pad 2: /LED2 -> /LED4
- P6 pad 1: /LED2 -> /LED4
- R17 pad 1: /LED3 -> /LED2
- R18 pad 1: /LED4 -> /LED3
Routing:
- net GND: track 116.4 -> 403.7 mm, vias 0 -> 3
- net +5V: track 48.0 -> 273.9 mm, vias 0 -> 9
- net /ENABLEB: track 0.00 -> 151.9 mm, vias 0 -> 2
- net /ENABLEA: track 0.00 -> 128.6 mm, vias 0 -> 2
- net /SENSOR 3: track 0.00 -> 120.8 mm, vias 0 -> 3
- net /IN_1A: track 0.00 -> 113.3 mm, vias 0 -> 2
- net /IN_2A: track 0.00 -> 103.2 mm, vias 0 -> 2
- net /SENSOR 2: track 0.00 -> 92.9 mm, vias 0 -> 4
- net /SENSOR 4: track 0.00 -> 85.4 mm, vias 0 -> 2
- net /LED4: track 0.00 -> 84.4 mm, vias 0 -> 2
- net /SENSOR 1: track 0.00 -> 71.4 mm, vias 0 -> 4
- net +BATT: track 0.00 -> 62.9 mm
- net +8V: track 6.51 -> 67.8 mm, vias 0 -> 2
- net /IN_3B: track 0.00 -> 48.5 mm, vias 0 -> 2
- net /LED3: track 0.00 -> 35.6 mm, vias 0 -> 1
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
Commit message: Terminado el ruteo! Incluidos los Gerber, drill, y Daiquiris de Frutilla
Parts:
- added P10: CONN_1, 1PIN2mm, F.Cu at (49.0, 111.1)
- added P11: CONN_1, 1PIN2mm, F.Cu at (46.0, 111.2)
- added P12: CONN_1, 1PIN2mm, F.Cu at (88.9, 85.7)
- added P13: CONN_1, 1PIN2mm, F.Cu at (41.2, 126.7)
- added P14: CONN_1, 1PIN2mm, F.Cu at (86.4, 83.5)
- added P15: CONN_1, 1PIN2mm, F.Cu at (37.1, 124.2)
- moved R1 212.5 mm to (272.9, 76.6)
- moved R2 212.5 mm to (256.9, 76.6)
- moved R8 212.5 mm to (271.9, 96.6)
- moved R9 212.5 mm to (256.9, 96.6)
- moved RV5 212.5 mm to (271.9, 93.6)
- moved RV6 212.5 mm to (256.9, 93.6)
- moved SERVO_U1 212.5 mm to (271.9, 86.6)
- moved SERVO_U2 212.5 mm to (256.9, 86.6)
Routing:
- net +5V: track 273.9 -> 481.1 mm, vias 9 -> 11
- net GND: track 403.7 -> 570.2 mm, vias 3 -> 6
- net +8V: track 67.8 -> 126.6 mm, vias 2 -> 3
- net /IN_1A: track 113.3 -> 149.1 mm
- net N-000007: track 25.4 -> 49.7 mm
- net /SENSOR 1: track 71.4 -> 95.7 mm
- net /SENSOR 2: track 92.9 -> 114.3 mm
- net /SCK: track 23.9 -> 42.1 mm
- net /SENSOR 3: track 120.8 -> 134.5 mm
- net /ENABLEB: track 151.9 -> 142.2 mm
- net N-0000054: track 52.5 -> 61.5 mm
- net N-0000021: track 13.7 -> 21.8 mm
- net /RX: track 11.2 -> 18.1 mm
- net /IN_2A: track 103.2 -> 108.9 mm
- net /ENABLEA: track 128.6 -> 123.6 mm
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- added copper zone on B.Cu, net (none)
- added copper zone on F.Cu, net (none)
Other:
- net class Default: trace_width 0.3048 -> 0.508
- board text added: "+5V"
- board text added: "3.14TITO"
- board text added: "GND"
- board text added: "LED 4"
- board text added: "SERVO"
- board text added: "sw"
