File: tito/Placa_Tito_2013/Placa_principal/placa_principal.sch (KiCad schematic (older format))
At the start: 67 parts, among them IC1 ATMEGA88-P, K1 Servo, K2 Jumper con doble posicion, P1 Puerto Serie, P2 Motor 1, P3 Motor 2, P4 Bateria 3,6V, P5 Bateria 7,2V, P6 Programador, P7 CONN_1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

Commit message: Liberadas interrupciones del micro para usar con futuros encoders, emprolijado esquematico
Parts:
- removed P8: JUMPERS PARA PROGRAMAR, symbol CONN_2X2
- added JP1, JP2: JUMPER, symbol JUMPER
- added P8, P9: CONN_1, symbol CONN_1
Connections:
- net labels removed: INTERRUPCION, PIN
- wire segments 244 -> 245
Other:
- note added: "Botones"
- note added: "Interrupciones\nlibres"
- note added: "Motores"
- moved on the sheet: C1, C2, C3, C7, C8, D1, D2, D3, D4, D5, D6, D7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

Commit message: Empezado el ruteo
Parts:
- renumbered U1 to SERVO_U1, U2 to SERVO_U2
Other:
- moved on the sheet: IC1

Commit message: Se terminaron de acomodar los componentes en la placa, y se inició el routeo de la misma
Parts:
- added JP3: JUMPER, symbol JUMPER
Connections:
- net SCK: now also JP3.1; no longer R3.2, SW1.1
- new net: JP3.2, R3.2, SW1.1
Changed lines of the file:
@@
-EESchema Schematic File Version 2  date vie 22 mar 2013 22:05:50 ART
+EESchema Schematic File Version 2  date vie 12 abr 2013 21:53:35 ART
 LIBS:power
 LIBS:device
@@
 Sheet 1 1
 Title "Tito, el autito más bonito"
-Date "23 mar 2013"
+Date "12 apr 2013"
 Rev "0.3"
 Comp ""
@@
 	1    0    0    -1
 $EndComp
-Text Label 8750 6650 0    60   ~ 0
+Text Label 7900 6650 2    60   ~ 0
 SWITCH
 $Comp
@@
 Text Notes 2000 2700 0    60   ~ 0
 Motores
+$Comp
+L JUMPER JP3
+U 1 1 516893DD
+P 8450 6650
+F 0 "JP3" H 8450 6800 60  0000 C CNN
+F 1 "JUMPER" H 8450 6570 40  0000 C CNN
+F 2 "" H 8450 6650 60  0001 C CNN
+F 3 "" H 8450 6650 60  0001 C CNN
+	1    8450 6650
+	1    0    0    -1
+$EndComp
+Wire Wire Line
+	8150 6650 7900 6650
 $EndSCHEMATC

Commit message: Casi finalizamos de routear la placa
Connections:
- net LED2: now also IC1.6 ((PCINT20/XCK/T0)PD4), R17.1; no longer IC1.18 ((PCINT4/MISO)PB4), JP2.2, P6.1
- net LED3: now also IC1.13 ((PCINT23/AIN1)PD7), R18.1; no longer IC1.6 ((PCINT20/XCK/T0)PD4), R17.1
- net LED4: now also IC1.18 ((PCINT4/MISO)PB4), JP2.2, P6.1; no longer IC1.13 ((PCINT23/AIN1)PD7), R18.1
- net SENSOR 1: now also IC1.26 ((PCINT11/ADC3)PC3); no longer IC1.23 ((PCINT8/ADC0)PC0)
- net SENSOR 2: now also IC1.25 ((PCINT10/ADC2)PC2); no longer IC1.24 ((PCINT9/ADC1)PC1)
- net SENSOR 3: now also IC1.24 ((PCINT9/ADC1)PC1); no longer IC1.25 ((PCINT10/ADC2)PC2)
- net SENSOR 4: now also IC1.23 ((PCINT8/ADC0)PC0); no longer IC1.26 ((PCINT11/ADC3)PC3)
Changed lines of the file:
@@
-EESchema Schematic File Version 2  date vie 12 abr 2013 21:53:35 ART
+EESchema Schematic File Version 2  date vie 19 abr 2013 21:08:42 ART
 LIBS:power
 LIBS:device
@@
 Sheet 1 1
 Title "Tito, el autito más bonito"
-Date "12 apr 2013"
+Date "20 apr 2013"
 Rev "0.3"
 Comp ""
@@
 Text Label 9850 3650 3    60   ~ 0
 LED1
+Text Label 10500 3700 3    60   ~ 0
+LED2
+Text Label 10800 3700 3    60   ~ 0
+LED3
 Text Label 10200 3100 3    60   ~ 0
-LED2
-Text Label 10500 3700 3    60   ~ 0
-LED3
-Text Label 10800 3700 3    60   ~ 0
 LED4
 $Comp
@@
 	1    0    0    -1
 $EndComp
+Text Label 3150 6350 2    60   ~ 0
+SENSOR 1
+Text Label 3150 6250 2    60   ~ 0
+SENSOR 2
+Text Label 3150 6150 2    60   ~ 0
+SENSOR 3
 Text Label 3150 6050 2    60   ~ 0
-SENSOR 1
-Text Label 3150 6150 2    60   ~ 0
-SENSOR 2
-Text Label 3150 6250 2    60   ~ 0
-SENSOR 3
-Text Label 3150 6350 2    60   ~ 0
 SENSOR 4
 Text Label 3150 6450 2    60   ~ 0
@@
 Text Label 2900 5200 2    60   ~ 0
 LED1
+Text Label 2900 7200 2    60   ~ 0
+LED2
+Text Label 2900 7500 2    60   ~ 0
+LED3
 Text Label 3500 5650 2    60   ~ 0
-LED2
-Text Label 2900 7200 2    60   ~ 0
-LED3
-Text Label 2900 7500 2    60   ~ 0
 LED4
 $Comp

Commit message: Terminado el ruteo! Incluidos los Gerber, drill, y Daiquiris de Frutilla
Parts:
- added P10, P11, P12, P13, P14, P15: CONN_1, ~, symbol CONN_1
Connections:
- net +5V: now also P12.1, P14.1
- net GND: now also P13.1, P15.1
- net SENSOR 5: now also P10.1
- net SENSOR 6: now also P11.1
Other:
- moved on the sheet: R1, R2, SERVO_U1, SERVO_U2
Changed lines of the file:
@@
-EESchema Schematic File Version 2  date vie 19 abr 2013 21:08:42 ART
+EESchema Schematic File Version 2  date vie 26 abr 2013 22:10:29 ART
 LIBS:power
 LIBS:device
@@
 Sheet 1 1
 Title "Tito, el autito más bonito"
-Date "20 apr 2013"
+Date "27 apr 2013"
 Rev "0.3"
 Comp ""
@@
 L CNY70 SERVO_U1
 U 1 1 50CBFFF7
-P 5750 1000
-F 0 "SERVO_U1" H 5750 1000 60  0000 C CNN
-F 1 "CNY70" H 5750 1000 60  0000 C CNN
-F 2 "" H 5750 1000 60  0001 C CNN
-F 3 "" H 5750 1000 60  0001 C CNN
-	1    5750 1000
+P 7150 1650
+F 0 "SERVO_U1" H 7150 1650 60  0000 C CNN
+F 1 "CNY70" H 7150 1650 60  0000 C CNN
+F 2 "" H 7150 1650 60  0001 C CNN
+F 3 "" H 7150 1650 60  0001 C CNN
+	1    7150 1650
 	1    0    0    -1
 $EndComp
@@
 L GND #PWR038
 U 1 1 50CBFFFD
-P 5300 1150
-F 0 "#PWR038" H 5300 1150 30  0001 C CNN
-F 1 "GND" H 5300 1080 30  0001 C CNN
-F 2 "" H 5300 1150 60  0001 C CNN
-F 3 "" H 5300 1150 60  0001 C CNN
-	1    5300 1150
+P 6700 1800
+F 0 "#PWR038" H 6700 1800 30  0001 C CNN
+F 1 "GND" H 6700 1730 30  0001 C CNN
+F 2 "" H 6700 1800 60  0001 C CNN
+F 3 "" H 6700 1800 60  0001 C CNN
+	1    6700 1800
 	1    0    0    -1
 $EndComp
@@
 L R R1
 U 1 1 50CC0004
-P 5700 700
-F 0 "R1" V 5780 700 50  0000 C CNN
-F 1 "R sensor" V 5700 700 50  0000 C CNN
-F 2 "" H 5700 700 60  0001 C CNN
-F 3 "" H 5700 700 60  0001 C CNN
-	1    5700 700
+P 7100 1350
+F 0 "R1" V 7180 1350 50  0000 C CNN
+F 1 "R sensor" V 7100 1350 50  0000 C CNN
+F 2 "" H 7100 1350 60  0001 C CNN
+F 3 "" H 7100 1350 60  0001 C CNN
+	1    7100 1350
 	0    -1   -1   0
 $EndComp
@@
 L +5V #PWR039
 U 1 1 50CC000A
-P 5950 650
-F 0 "#PWR039" H 5950 740 20  0001 C CNN
-F 1 "+5V" H 5950 740 30  0000 C CNN
-F 2 "" H 5950 650 60  0001 C CNN
-F 3 "" H 5950 650 60  0001 C CNN
-	1    5950 650
-	1    0    0    -1
-$EndComp
-Text Label 6500 1100 2    60   ~ 0
+P 7350 1300
+F 0 "#PWR039" H 7350 1390 20  0001 C CNN
+F 1 "+5V" H 7350 1390 30  0000 C CNN
+F 2 "" H 7350 1300 60  0001 C CNN
+F 3 "" H 7350 1300 60  0001 C CNN
+	1    7350 1300
+	1    0    0    -1
+$EndComp
+Text Label 7900 1750 2    60   ~ 0
 SENSOR 5
 $Comp
 L CNY70 SERVO_U2
 U 1 1 50CC0019
-P 5750 1650
-F 0 "SERVO_U2" H 5750 1650 60  0000 C CNN
-F 1 "CNY70" H 5750 1650 60  0000 C CNN
-F 2 "" H 5750 1650 60  0001 C CNN
-F 3 "" H 5750 1650 60  0001 C CNN
-	1    5750 1650
+P 7150 2300
+F 0 "SERVO_U2" H 7150 2300 60  0000 C CNN
+F 1 "CNY70" H 7150 2300 60  0000 C CNN
+F 2 "" H 7150 2300 60  0001 C CNN
+F 3 "" H 7150 2300 60  0001 C CNN
+	1    7150 2300
 	1    0    0    -1
 $EndComp
@@
 L GND #PWR040
 U 1 1 50CC001F
-P 5300 1800
-F 0 "#PWR040" H 5300 1800 30  0001 C CNN
-F 1 "GND" H 5300 1730 30  0001 C CNN
-F 2 "" H 5300 1800 60  0001 C CNN
-F 3 "" H 5300 1800 60  0001 C CNN
-	1    5300 1800
+P 6700 2450
+F 0 "#PWR040" H 6700 2450 30  0001 C CNN
+F 1 "GND" H 6700 2380 30  0001 C CNN
+F 2 "" H 6700 2450 60  0001 C CNN
+F 3 "" H 6700 2450 60  0001 C CNN
+	1    6700 2450
 	1    0    0    -1
 $EndComp
@@
 L R R2
 U 1 1 50CC0026
-P 5700 1350
-F 0 "R2" V 5780 1350 50  0000 C CNN
-F 1 "R sensor" V 5700 1350 50  0000 C CNN
-F 2 "" H 5700 1350 60  0001 C CNN
-F 3 "" H 5700 1350 60  0001 C CNN
-	1    5700 1350
+P 7100 2000
+F 0 "R2" V 7180 2000 50  0000 C CNN
+F 1 "R sensor" V 7100 2000 50  0000 C CNN
+F 2 "" H 7100 2000 60  0001 C CNN
+F 3 "" H 7100 2000 60  0001 C CNN
+	1    7100 2000
 	0    -1   -1   0
 $EndComp
@@
 L +5V #PWR041
 U 1 1 50CC002C
-P 5950 1300
-F 0 "#PWR041" H 5950 1390 20  0001 C CNN
-F 1 "+5V" H 5950 1390 30  0000 C CNN
-F 2 "" H 5950 1300 60  0001 C CNN
-F 3 "" H 5950 1300 60  0001 C CNN
-	1    5950 1300
-	1    0    0    -1
-$EndComp
-Text Label 6500 1750 2    60   ~ 0
+P 7350 1950
+F 0 "#PWR041" H 7350 2040 20  0001 C CNN
+F 1 "+5V" H 7350 2040 30  0000 C CNN
+F 2 "" H 7350 1950 60  0001 C CNN
+F 3 "" H 7350 1950 60  0001 C CNN
+	1    7350 1950
+	1    0    0    -1
+$EndComp
+Text Label 7900 2400 2    60   ~ 0
 SENSOR 6
 $Comp
@@
 	900  2050 800  2050
 Wire Wire Line
-	5300 1750 5350 1750
-Wire Wire Line
-	5300 1800 5300 1750
-Connection ~ 5950 1350
-Wire Wire Line
-	5350 1350 5350 1550
-Wire Wire Line
-	5450 1350 5350 1350
-Wire Wire Line
-	6050 1350 5950 1350
-Wire Wire Line
-	6050 1550 6050 1350
-Wire Wire Line
-	5950 1350 5950 1300
-Wire Wire Line
-	6050 1750 6500 1750
-Wire Wire Line
-	5300 1100 5350 1100
-Wire Wire Line
-	5300 1150 5300 1100
-Connection ~ 5950 700
-Wire Wire Line
-	5350 700  5350 900
-Wire Wire Line
-	5450 700  5350 700
-Wire Wire Line
-	6050 700  5950 700
-Wire Wire Line
-	6050 900  6050 700
-Wire Wire Line
-	5950 700  5950 650
-Wire Wire Line
-	6050 1100 6500 1100
+	6700 2400 6750 2400
+Wire Wire Line
+	6700 2450 6700 2400
+Connection ~ 7350 2000
+Wire Wire Line
+	6750 2000 6750 2200
+Wire Wire Line
+	6850 2000 6750 2000
+Wire Wire Line
+	7450 2000 7350 2000
+Wire Wire Line
+	7450 2200 7450 2000
+Wire Wire Line
+	7350 2000 7350 1950
+Wire Wire Line
+	7450 2400 7950 2400
+Wire Wire Line
+	6700 1750 6750 1750
+Wire Wire Line
+	6700 1800 6700 1750
+Connection ~ 7350 1350
+Wire Wire Line
+	6750 1350 6750 1550
+Wire Wire Line
+	6850 1350 6750 1350
+Wire Wire Line
+	7450 1350 7350 1350
+Wire Wire Line
+	7450 1550 7450 1350
+Wire Wire Line
+	7350 1350 7350 1300
+Wire Wire Line
+	7450 1750 7950 1750
 Wire Wire Line
 	2700 5300 2950 5300
@@
 	750  5150 750  5500
 Wire Wire Line
-	800  5200 750  5200
+	550  5200 800  5200
 Connection ~ 700  7500
 Wire Wire Line
 	800  7500 700  7500
 Wire Wire Line
-	700  7400 700  7600
+	700  7350 700  7600
 Wire Wire Line
 	800  7400 700  7400
@@
 Wire Wire Line
 	8150 6650 7900 6650
+$Comp
+L CONN_1 P10
+U 1 1 517B01FC
+P 7950 1600
+F 0 "P10" H 8030 1600 40  0000 L CNN
+F 1 "CONN_1" H 7950 1655 30  0001 C CNN
+F 2 "~" H 7950 1600 60  0000 C CNN
+F 3 "~" H 7950 1600 60  0000 C CNN
+	1    7950 1600
+	0    -1   -1   0
+$EndComp
+$Comp
+L CONN_1 P11
+U 1 1 517B020B
+P 7950 2250
+F 0 "P11" H 8030 2250 40  0000 L CNN
+F 1 "CONN_1" H 7950 2305 30  0001 C CNN
+F 2 "~" H 7950 2250 60  0000 C CNN
+F 3 "~" H 7950 2250 60  0000 C CNN
+	1    7950 2250
+	0    -1   -1   0
+$EndComp
+$Comp
+L CONN_1 P15
+U 1 1 517B2049
+P 700 7200
+F 0 "P15" H 780 7200 40  0000 L CNN
+F 1 "CONN_1" H 700 7255 30  0001 C CNN
+F 2 "~" H 700 7200 60  0000 C CNN
+F 3 "~" H 700 7200 60  0000 C CNN
+	1    700  7200
+	0    -1   -1   0
+$EndComp
+$Comp
+L CONN_1 P13
+U 1 1 517B2056
+P 600 7200
+F 0 "P13" H 680 7200 40  0000 L CNN
+F 1 "CONN_1" H 600 7255 30  0001 C CNN
+F 2 "~" H 600 7200 60  0000 C CNN
+F 3 "~" H 600 7200 60  0000 C CNN
+	1    600  7200
+	0    -1   -1   0
+$EndComp
+Wire Wire Line
+	600  7350 700  7350
+Connection ~ 700  7400
+$Comp
+L CONN_1 P14
+U 1 1 517B2301
+P 650 5050
+F 0 "P14" H 730 5050 40  0000 L CNN
+F 1 "CONN_1" H 650 5105 30  0001 C CNN
+F 2 "~" H 650 5050 60  0000 C CNN
+F 3 "~" H 650 5050 60  0000 C CNN
+	1    650  5050
+	0    -1   -1   0
+$EndComp
+$Comp
+L CONN_1 P12
+U 1 1 517B2315
+P 550 5050
+F 0 "P12" H 630 5050 40  0000 L CNN
+F 1 "CONN_1" H 550 5105 30  0001 C CNN
+F 2 "~" H 550 5050 60  0000 C CNN
+F 3 "~" H 550 5050 60  0000 C CNN
+	1    550  5050
+	0    -1   -1   0
+$EndComp
+Connection ~ 650  5200
 $EndSCHEMATC
