File: Placas/Placa_Tito_2013/Placa_principal/placa_principal.sch (KiCad schematic (older format))
At the start: 77 parts, among them IC1 ATMEGA88-P, K1 Servo, K2 Jumper con doble posicion, P1 Puerto Serie, P10 CONN_1, P11 CONN_1, P12 CONN_1, P13 CONN_1, P14 CONN_1, P15 CONN_1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

Commit message: Agrego las bibliotecas del tcrt1000, y cambio los componentes en el esquemático
Parts:
- removed SERVO_U1, SERVO_U2, U3, U4, U6, U7: CNY70, symbol CNY70
- added U? (x6): TCRT1000, TCRT1000, symbol TCRT1000
Connections:
- wire segments 247 -> 235
Other:
- moved on the sheet: P10, P11

Commit message: Se termino de routear la placa con los nuevos sensores
Parts:
- gave numbers to parts that had none: 6

Commit message: Agrego hoja de datos del BC548C, y realizo cambios propuestos sobre el esquematico de la placa
Parts:
- removed K2: Jumper con doble posicion, symbol CONN_3
- removed P7: CONN_1, symbol CONN_1
- added C?: 10 nF, symbol C
- added C?: 220 uF, symbol CAPAPOL
- added C? (x2): 15 Pf, symbol C
- added Q?: BC548, TO92, symbol BC548
- added SW? (x2): DUAL_SWITCH_INV, symbol DUAL_SWITCH_INV
- added U?: REG_104-3, symbol REG_104-5
- added X?: 12 MHz, symbol CRYSTAL
Connections:
- net labels added: +3,3V, Habilitador Sensores, Pin Habilitador, Xtal1, Xtal2
- net labels removed: ENABLEA, ENABLEB
- wire segments 235 -> 271
Other:
- note added: "Regulador de tension de 5V y 3,3V\n"
- note removed: "Regulador de tension\n"
- moved on the sheet: C6, D10, D11, D12, D9, JP2, P10, P11, P5, P6, R1, R10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

Commit message: Agregado cristal externo
Parts:
- U?: value REG_104-3 -> REG_104-3.3
Changed lines of the file:
@@
 P 10000 2550
 F 0 "U?" H 9750 2750 60  0000 C CNN
-F 1 "REG_104-3" H 10000 2850 60  0000 C CNN
+F 1 "REG_104-3.3" H 10000 2850 60  0000 C CNN
 F 2 "" H 10000 2550 60  0001 C CNN
 F 3 "" H 10000 2550 60  0001 C CNN

Commit message: Empezados conversores 5V a 3,3V y viceversa en esquemático.
Parts:
- added 17k, 33k: R, ~, symbol R
- X?: value 12 MHz -> 18,432 MHz
Connections:
- wire segments 271 -> 277
Other:
- note added: "5 a 3,3\n3,3 a 5"
Changed lines of the file:
@@
 LIBS:tcrt1000
 LIBS:placa_principal-cache
-EELAYER 24 0
+EELAYER 27 0
 EELAYER END
 $Descr A4 11693 8268
@@
 Sheet 1 1
 Title "Tito, el autito más bonito"
-Date "12 jul 2013"
+Date "7 mar 2014"
 Rev "0.3"
 Comp ""
@@
 P 6350 2300
 F 0 "X?" H 6350 2450 60  0000 C CNN
-F 1 "12 MHz" H 6350 2150 60  0000 C CNN
+F 1 "18,432 MHz" H 6350 2150 60  0000 C CNN
 F 2 "" H 6350 2300 60  0000 C CNN
 F 3 "" H 6350 2300 60  0000 C CNN
@@
 Wire Wire Line
 	9250 2450 9500 2450
+$Comp
+L +5V #PWR?
+U 1 1 531A2D0E
+P 10450 3900
+F 0 "#PWR?" H 10450 3990 20  0001 C CNN
+F 1 "+5V" H 10450 3990 30  0000 C CNN
+F 2 "" H 10450 3900 60  0000 C CNN
+F 3 "" H 10450 3900 60  0000 C CNN
+	1    10450 3900
+	1    0    0    -1
+$EndComp
+$Comp
+L +3,3V #PWR?
+U 1 1 531A2D1D
+P 11100 3900
+F 0 "#PWR?" H 11100 3860 30  0001 C CNN
+F 1 "+3,3V" H 11100 4010 30  0000 C CNN
+F 2 "" H 11100 3900 60  0000 C CNN
+F 3 "" H 11100 3900 60  0000 C CNN
+	1    11100 3900
+	1    0    0    -1
+$EndComp
+$Comp
+L R 17k
+U 1 1 531A2D2C
+P 10750 3950
+F 0 "17k" V 10830 3950 40  0000 C CNN
+F 1 "R" V 10757 3951 40  0000 C CNN
+F 2 "~" V 10680 3950 30  0000 C CNN
+F 3 "~" H 10750 3950 30  0000 C CNN
+	1    10750 3950
+	0    -1   -1   0
+$EndComp
+$Comp
+L R 33k
+U 1 1 531A2D3B
+P 11050 4250
+F 0 "33k" V 11130 4250 40  0000 C CNN
+F 1 "R" V 11057 4251 40  0000 C CNN
+F 2 "~" V 10980 4250 30  0000 C CNN
+F 3 "~" H 11050 4250 30  0000 C CNN
+	1    11050 4250
+	1    0    0    -1
+$EndComp
+$Comp
+L GND #PWR?
+U 1 1 531A2D4A
+P 11050 4550
+F 0 "#PWR?" H 11050 4550 30  0001 C CNN
+F 1 "GND" H 11050 4480 30  0001 C CNN
+F 2 "" H 11050 4550 60  0000 C CNN
+F 3 "" H 11050 4550 60  0000 C CNN
+	1    11050 4550
+	1    0    0    -1
+$EndComp
+Wire Wire Line
+	11000 3950 11050 3950
+Wire Wire Line
+	11050 3900 11050 4000
+Wire Wire Line
+	10500 3950 10450 3950
+Wire Wire Line
+	10450 3950 10450 3900
+Wire Wire Line
+	11100 3900 11050 3900
+Connection ~ 11050 3950
+Wire Wire Line
+	11050 4500 11050 4550
+Text Notes 10600 4200 0    60   ~ 0
+5 a 3,3\n3,3 a 5
 $EndSCHEMATC

Commit message: Creo y agrego el esquematico de nuestro nuevo puente H (DRV8833), falta corregir ruta de la biblioteca
Parts:
- added U?: DRV8833, ~, symbol DRV8833
Changed lines of the file:
@@
 LIBS:cny70
 LIBS:tcrt1000
-LIBS:placa_principal-cache
+LIBS:drv8833
 EELAYER 27 0
 EELAYER END
@@
 Sheet 1 1
 Title "Tito, el autito más bonito"
-Date "7 mar 2014"
+Date "12 may 2014"
 Rev "0.3"
 Comp ""
@@
 Text Notes 10600 4200 0    60   ~ 0
 5 a 3,3\n3,3 a 5
+$Comp
+L DRV8833 U?
+U 1 1 53714B04
+P 5800 1250
+F 0 "U?" H 5850 1600 60  0000 C CNN
+F 1 "DRV8833" H 5800 1700 60  0000 C CNN
+F 2 "~" H 5800 1250 60  0000 C CNN
+F 3 "~" H 5800 1250 60  0000 C CNN
+	1    5800 1250
+	1    0    0    -1
+$EndComp
 $EndSCHEMATC

Commit message: Empezados cambios en esquemático para puente H SMD, DRV8833. Agregado datasheet del mismo al repo.
Parts:
- removed IC1: ATMEGA88-P, DIL28, symbol ATMEGA88-P
- added IC?: ATMEGA88A-A, TQFP32, symbol ATMEGA88A-A
- added R?: R, ~, symbol R
Connections:
- net labels added: VCC
- wire segments 277 -> 286
Other:
- moved on the sheet: C?
Changed lines of the file:
@@
 LIBS:tcrt1000
 LIBS:drv8833
+LIBS:placa_principal-cache
 EELAYER 27 0
 EELAYER END
@@
 Sheet 1 1
 Title "Tito, el autito más bonito"
-Date "12 may 2014"
+Date "16 may 2014"
 Rev "0.3"
 Comp ""
@@
 $EndComp
 $Comp
-L ATMEGA88-P IC1
-U 1 1 50A703EB
-P 1800 6350
-F 0 "IC1" H 1100 7600 50  0000 L BNN
-F 1 "ATMEGA88-P" H 2100 4950 50  0000 L BNN
-F 2 "DIL28" H 1200 5000 50  0001 C CNN
-F 3 "" H 1800 6350 60  0001 C CNN
-	1    1800 6350
-	1    0    0    -1
-$EndComp
-$Comp
 L LED D9
 U 1 1 50A70BBD
@@
 	1    0    0    -1
 $EndComp
-Text Notes 4650 650  2    60   ~ 0
+Text Notes 4700 600  2    60   ~ 0
 Leds de control\n
 Text Notes 9250 950  0    60   ~ 0
@@
 L CRYSTAL X?
 U 1 1 52FEBA3F
-P 6350 2300
-F 0 "X?" H 6350 2450 60  0000 C CNN
-F 1 "18,432 MHz" H 6350 2150 60  0000 C CNN
-F 2 "" H 6350 2300 60  0000 C CNN
-F 3 "" H 6350 2300 60  0000 C CNN
-	1    6350 2300
+P 9600 5000
+F 0 "X?" H 9600 5150 60  0000 C CNN
+F 1 "18,432 MHz" H 9600 4850 60  0000 C CNN
+F 2 "" H 9600 5000 60  0000 C CNN
+F 3 "" H 9600 5000 60  0000 C CNN
+	1    9600 5000
 	1    0    0    -1
 $EndComp
@@
 L C C?
 U 1 1 52FEBA4E
-P 6000 2550
-F 0 "C?" H 6000 2650 40  0000 L CNN
-F 1 "15 Pf" H 6006 2465 40  0000 L CNN
-F 2 "" H 6038 2400 30  0000 C CNN
-F 3 "" H 6000 2550 60  0000 C CNN
-	1    6000 2550
+P 9250 5250
+F 0 "C?" H 9250 5350 40  0000 L CNN
+F 1 "15 Pf" H 9256 5165 40  0000 L CNN
+F 2 "" H 9288 5100 30  0000 C CNN
+F 3 "" H 9250 5250 60  0000 C CNN
+	1    9250 5250
 	1    0    0    -1
 $EndComp
@@
 L C C?
 U 1 1 52FEBA5D
-P 6700 2550
-F 0 "C?" H 6700 2650 40  0000 L CNN
-F 1 "15 Pf" H 6706 2465 40  0000 L CNN
-F 2 "" H 6738 2400 30  0000 C CNN
-F 3 "" H 6700 2550 60  0000 C CNN
-	1    6700 2550
+P 9950 5250
+F 0 "C?" H 9950 5350 40  0000 L CNN
+F 1 "15 Pf" H 9956 5165 40  0000 L CNN
+F 2 "" H 9988 5100 30  0000 C CNN
+F 3 "" H 9950 5250 60  0000 C CNN
+	1    9950 5250
 	1    0    0    -1
 $EndComp
@@
 L GND #PWR?
 U 1 1 52FEC00C
-P 6350 2800
-F 0 "#PWR?" H 6350 2800 30  0001 C CNN
-F 1 "GND" H 6350 2730 30  0001 C CNN
-F 2 "" H 6350 2800 60  0000 C CNN
-F 3 "" H 6350 2800 60  0000 C CNN
-	1    6350 2800
-	1    0    0    -1
-$EndComp
-Text Label 6000 2050 0    60   ~ 0
+P 9600 5500
+F 0 "#PWR?" H 9600 5500 30  0001 C CNN
+F 1 "GND" H 9600 5430 30  0001 C CNN
+F 2 "" H 9600 5500 60  0000 C CNN
+F 3 "" H 9600 5500 60  0000 C CNN
+	1    9600 5500
+	1    0    0    -1
+$EndComp
+Text Label 9250 4750 0    60   ~ 0
 Xtal1
-Text Label 6700 2050 2    60   ~ 0
+Text Label 9950 4750 2    60   ~ 0
 Xtal2
 Text Label 3350 7000 2    60   ~ 0
@@
 	1    8750 1650
 	-1   0    0    1
+$EndComp
+$Comp
+L DUAL_SWITCH_INV SW?
+U 1 1 52FEDED8
+P 8750 2800
+F 0 "SW?" H 8550 2950 50  0000 C CNN
+F 1 "DUAL_SWITCH_INV" H 8600 2650 50  0000 C CNN
+F 2 "" H 8750 2800 60  0000 C CNN
+F 3 "" H 8750 2800 60  0000 C CNN
+	1    8750 2800
+	-1   0    0    1
+$EndComp
+$Comp
+L +5V #PWR?
+U 1 1 531A2D0E
+P 10450 3900
+F 0 "#PWR?" H 10450 3990 20  0001 C CNN
+F 1 "+5V" H 10450 3990 30  0000 C CNN
+F 2 "" H 10450 3900 60  0000 C CNN
+F 3 "" H 10450 3900 60  0000 C CNN
+	1    10450 3900
+	1    0    0    -1
+$EndComp
+$Comp
+L +3,3V #PWR?
+U 1 1 531A2D1D
+P 11100 3900
+F 0 "#PWR?" H 11100 3860 30  0001 C CNN
+F 1 "+3,3V" H 11100 4010 30  0000 C CNN
+F 2 "" H 11100 3900 60  0000 C CNN
+F 3 "" H 11100 3900 60  0000 C CNN
+	1    11100 3900
+	1    0    0    -1
+$EndComp
+$Comp
+L R 17k
+U 1 1 531A2D2C
+P 10750 3950
+F 0 "17k" V 10830 3950 40  0000 C CNN
+F 1 "R" V 10757 3951 40  0000 C CNN
+F 2 "~" V 10680 3950 30  0000 C CNN
+F 3 "~" H 10750 3950 30  0000 C CNN
+	1    10750 3950
+	0    -1   -1   0
+$EndComp
+$Comp
+L R 33k
+U 1 1 531A2D3B
+P 11050 4250
+F 0 "33k" V 11130 4250 40  0000 C CNN
+F 1 "R" V 11057 4251 40  0000 C CNN
+F 2 "~" V 10980 4250 30  0000 C CNN
+F 3 "~" H 11050 4250 30  0000 C CNN
+	1    11050 4250
+	1    0    0    -1
+$EndComp
+$Comp
+L GND #PWR?
+U 1 1 531A2D4A
+P 11050 4550
+F 0 "#PWR?" H 11050 4550 30  0001 C CNN
+F 1 "GND" H 11050 4480 30  0001 C CNN
+F 2 "" H 11050 4550 60  0000 C CNN
+F 3 "" H 11050 4550 60  0000 C CNN
+	1    11050 4550
+	1    0    0    -1
+$EndComp
+Text Notes 10600 4200 0    60   ~ 0
+5 a 3,3\n3,3 a 5
+$Comp
+L DRV8833 U?
+U 1 1 53714B04
+P 6700 2350
+F 0 "U?" H 6750 2700 60  0000 C CNN
+F 1 "DRV8833" H 6700 2800 60  0000 C CNN
+F 2 "~" H 6700 2350 60  0000 C CNN
+F 3 "~" H 6700 2350 60  0000 C CNN
+	1    6700 2350
+	1    0    0    -1
+$EndComp
+$Comp
+L ATMEGA88A-A IC?
+U 1 1 53769604
+P 1700 6300
+F 0 "IC?" H 950 7550 40  0000 L BNN
+F 1 "ATMEGA88A-A" H 2100 4900 40  0000 L BNN
+F 2 "TQFP32" H 1700 6300 30  0000 C CIN
+F 3 "" H 1700 6300 60  0000 C CNN
+	1    1700 6300
+	1    0    0    -1
 $EndComp
 Wire Wire Line
@@
 Wire Wire Line
 	1500 4300 1200 4300
-Connection ~ 13050 9050
 Wire Wire Line
 	1200 4000 1500 4000
@@
 	5200 6550 5150 6550
 Wire Wire Line
-	6000 2050 6000 2350
-Wire Wire Line
-	6000 2300 6050 2300
-Wire Wire Line
-	6650 2300 6700 2300
-Wire Wire Line
-	6700 2050 6700 2350
-Wire Wire Line
-	6000 2750 6700 2750
-Wire Wire Line
-	6350 2750 6350 2800
-Connection ~ 6350 2750
-Connection ~ 6000 2300
-Connection ~ 6700 2300
+	9250 4750 9250 5050
+Wire Wire Line
+	9250 5000 9300 5000
+Wire Wire Line
+	9900 5000 9950 5000
+Wire Wire Line
+	9950 4750 9950 5050
+Wire Wire Line
+	9250 5450 9950 5450
+Wire Wire Line
+	9600 5450 9600 5500
+Connection ~ 9600 5450
+Connection ~ 9250 5000
+Connection ~ 9950 5000
 Wire Wire Line
 	2700 5900 2950 5900
@@
 Wire Wire Line
 	8300 1300 8300 1250
-$Comp
-L DUAL_SWITCH_INV SW?
-U 1 1 52FEDED8
-P 8750 2800
-F 0 "SW?" H 8550 2950 50  0000 C CNN
-F 1 "DUAL_SWITCH_INV" H 8600 2650 50  0000 C CNN
-F 2 "" H 8750 2800 60  0000 C CNN
-F 3 "" H 8750 2800 60  0000 C CNN
-	1    8750 2800
-	-1   0    0    1
-$EndComp
 Wire Wire Line
 	8250 2900 8250 3000
@@
 Wire Wire Line
 	9250 2450 9500 2450
-$Comp
-L +5V #PWR?
-U 1 1 531A2D0E
-P 10450 3900
-F 0 "#PWR?" H 10450 3990 20  0001 C CNN
-F 1 "+5V" H 10450 3990 30  0000 C CNN
-F 2 "" H 10450 3900 60  0000 C CNN
-F 3 "" H 10450 3900 60  0000 C CNN
-	1    10450 3900
-	1    0    0    -1
-$EndComp
-$Comp
-L +3,3V #PWR?
-U 1 1 531A2D1D
-P 11100 3900
-F 0 "#PWR?" H 11100 3860 30  0001 C CNN
-F 1 "+3,3V" H 11100 4010 30  0000 C CNN
-F 2 "" H 11100 3900 60  0000 C CNN
-F 3 "" H 11100 3900 60  0000 C CNN
-	1    11100 3900
-	1    0    0    -1
-$EndComp
-$Comp
-L R 17k
-U 1 1 531A2D2C
-P 10750 3950
-F 0 "17k" V 10830 3950 40  0000 C CNN
-F 1 "R" V 10757 3951 40  0000 C CNN
-F 2 "~" V 10680 3950 30  0000 C CNN
-F 3 "~" H 10750 3950 30  0000 C CNN
-	1    10750 3950
-	0    -1   -1   0
-$EndComp
-$Comp
-L R 33k
-U 1 1 531A2D3B
-P 11050 4250
-F 0 "33k" V 11130 4250 40  0000 C CNN
-F 1 "R" V 11057 4251 40  0000 C CNN
-F 2 "~" V 10980 4250 30  0000 C CNN
-F 3 "~" H 11050 4250 30  0000 C CNN
-	1    11050 4250
-	1    0    0    -1
-$EndComp
-$Comp
-L GND #PWR?
-U 1 1 531A2D4A
-P 11050 4550
-F 0 "#PWR?" H 11050 4550 30  0001 C CNN
-F 1 "GND" H 11050 4480 30  0001 C CNN
-F 2 "" H 11050 4550 60  0000 C CNN
-F 3 "" H 11050 4550 60  0000 C CNN
-	1    11050 4550
-	1    0    0    -1
-$EndComp
 Wire Wire Line
 	11000 3950 11050 3950
@@
 Wire Wire Line
 	11050 4500 11050 4550
-Text Notes 10600 4200 0    60   ~ 0
-5 a 3,3\n3,3 a 5
-$Comp
-L DRV8833 U?
-U 1 1 53714B04
-P 5800 1250
-F 0 "U?" H 5850 1600 60  0000 C CNN
-F 1 "DRV8833" H 5800 1700 60  0000 C CNN
-F 2 "~" H 5800 1250 60  0000 C CNN
-F 3 "~" H 5800 1250 60  0000 C CNN
-	1    5800 1250
-	1    0    0    -1
-$EndComp
+Wire Wire Line
+	800  5300 750  5300
+Connection ~ 750  5300
+Wire Wire Line
+	6000 2500 5600 2500
+Wire Wire Line
+	6000 2200 5600 2200
+Wire Wire Line
+	5600 2200 5600 2250
+$Comp
+L GND #PWR?
+U 1 1 5376A167
+P 5600 2250
+F 0 "#PWR?" H 5600 2250 30  0001 C CNN
+F 1 "GND" H 5600 2180 30  0001 C CNN
+F 2 "" H 5600 2250 60  0000 C CNN
+F 3 "" H 5600 2250 60  0000 C CNN
+	1    5600 2250
+	1    0    0    -1
+$EndComp
+$Comp
+L GND #PWR?
+U 1 1 5376A176
+P 5600 2500
+F 0 "#PWR?" H 5600 2500 30  0001 C CNN
+F 1 "GND" H 5600 2430 30  0001 C CNN
+F 2 "" H 5600 2500 60  0000 C CNN
+F 3 "" H 5600 2500 60  0000 C CNN
+	1    5600 2500
+	1    0    0    -1
+$EndComp
+$Comp
+L VCC #PWR?
+U 1 1 5376A185
+P 5750 1400
+F 0 "#PWR?" H 5750 1500 30  0001 C CNN
+F 1 "VCC" H 5750 1500 30  0000 C CNN
+F 2 "" H 5750 1400 60  0000 C CNN
+F 3 "" H 5750 1400 60  0000 C CNN
+	1    5750 1400
+	1    0    0    -1
+$EndComp
+Wire Wire Line
+	5750 2000 6000 2000
+Wire Wire Line
+	5750 2000 5750 1950
+$Comp
+L R R?
+U 1 1 5376A491
+P 5750 1700
+F 0 "R?" V 5830 1700 40  0000 C CNN
+F 1 "R" V 5757 1701 40  0000 C CNN
+F 2 "~" V 5680 1700 30  0000 C CNN
+F 3 "~" H 5750 1700 30  0000 C CNN
+	1    5750 1700
+	1    0    0    -1
+$EndComp
+Wire Wire Line
+	5750 1450 5750 1400
+Wire Wire Line
+	7400 2300 7750 2300
+Wire Wire Line
+	7750 2300 7750 2350
+$Comp
+L GND #PWR?
+U 1 1 5376A968
+P 7750 2350
+F 0 "#PWR?" H 7750 2350 30  0001 C CNN
+F 1 "GND" H 7750 2280 30  0001 C CNN
+F 2 "" H 7750 2350 60  0000 C CNN
+F 3 "" H 7750 2350 60  0000 C CNN
+	1    7750 2350
+	1    0    0    -1
+$EndComp

Commit message: Separadas partes del esquématico en varias hojas. Ajustes al esquemático.
Parts:
- removed C1: 100 nF, symbol C
- removed C2: 1000 uF, symbol CAPAPOL
- removed C4, C?: 220 uF, symbol CAPAPOL
- removed C5, C?: 10 nF, symbol C
- removed C6: 100nF, symbol C
- removed C7: 100uF, symbol CAPAPOL
- removed D1, D2, D3, D4, D5, D6, D7, D8: DIODE, symbol DIODE
- removed JP2: JUMPER, symbol JUMPER
- removed K1: Servo, symbol CONN_3
- removed P10, P11: CONN_1, ~, symbol CONN_1
- removed P2: Motor 1, symbol CONN_2
- removed P3: Motor 2, symbol CONN_2
- removed P4: Bateria 3,6V, symbol CONN_2
- removed P5: Bateria 7,2V, symbol CONN_2
- removed P8: CONN_1, symbol CONN_1
- removed R1, R10, R11, R12, R13, R2: R sensor, symbol R
- removed R4, R5, R6, R7, R8, R9: 100, symbol R
- removed R?: R, ~, symbol R
- removed RV1, RV2, RV3, RV4, RV5, RV6: POT, symbol POT
- removed SERVO_U1, SERVO_U2, U3, U4, U6, U7: TCRT1000, TCRT1000, symbol TCRT1000
- removed SW? (x2): DUAL_SWITCH_INV, symbol DUAL_SWITCH_INV
- removed U5: L298D, symbol L298D
- removed U8: REG_104-5, symbol REG_104-5
- removed U?: REG_104-3.3, symbol REG_104-5
- removed U?: DRV8833, ~, symbol DRV8833
- added JP? (x2): JUMPER, symbol JUMPER
- gave numbers to parts that had none: 5
- renumbered 17k to 17k1, 33k to 33k1
Connections:
- net labels added: +3.3V, IN_1B, IN_2B, VDD
- net labels removed: +8V, IN_3B, IN_4B, MOT_1A, MOT_2A, MOT_3B, MOT_4B, VCC
- wire segments 286 -> 154
Other:
- note added: "Alimentación"
- note added: "Sensores"
- note removed: "10.8 V"
- note removed: "Interrupciones\nlibres"
- note removed: "Regulador de tension de 5V y 3,3V\n"
- note removed: "Resistencias\nde seguridad"
- moved on the sheet: 17k1, 33k1, C11, C3, C8, C9, D10, D11, D12, D9, JP1, JP3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
