File: Placas/Placa_Tito_2013/Placa_principal/placa_principal.sch (KiCad schematic (older format))
At the start: 34 parts, among them IC1 ATMEGA88A-A, P1 Puerto Serie, P12 CONN_1, P13 CONN_1, P14 CONN_1, P15 CONN_1, P6 Programador, P9 CONN_1, Q1 BC548, SW1 SWITCH COMUN, SW2 SW_PUSH_SMALL, SW3 BOTON DE INTERRUPCION, X1 18,432 MHz

Commit message: Ajustes de estandarización de nombres en componentes y etiquetas del esquemático. Removido cny70 del .pro, agregado datasheet tcrt1000
Parts:
- removed 17k1, 33k1: R, ~, symbol R
- C11, C9: value 15 Pf -> 15 p
- JP1, JP? (x2): value JUMPER -> PUENTE
- R15, R16, R17, R18: value R led -> 220
- X1: value 18,432 MHz -> 18,432 M
Connections:
- net labels added: HABILITADOR SENSORES, PIN HABILITADOR
- net labels removed: Habilitador Sensores, Pin Habilitador
- wire segments 154 -> 129
Other:
- note removed: "5 a 3,3\n3,3 a 5"

Commit message: Terminado esquemático. Comenzado a asociar componentes.
Parts:
- removed JP3: JUMPER, symbol JUMPER
- removed P9: CONN_1, symbol CONN_1
- C1: renamed from C8; value 100nF -> 100n
- C4: renamed from C3; value 100n -> 100 n
- JP1: value PUENTE -> PUENTE FALLBACK
- JP2, JP3: renamed from JP?; value PUENTE -> PUENTE FALLBACK
- P1: renamed from P12; value CONN_1 -> ADICIONAL 5V
- P2: renamed from P13; value CONN_1 -> ADICIONAL GND
- P3: renamed from P14; value CONN_1 -> ADICIONAL 5V
- P4: renamed from P15; value CONN_1 -> ADICIONAL GND
- R5: renamed from R3; value PULL UP -> 10 k
- R6: renamed from R19; value PULL UP -> 10 k
- SW1: value SWITCH COMUN -> BOTÓN 1
- SW2: renamed from SW3; value BOTON DE INTERRUPCION -> BOTÓN 2
- SW3: renamed from SW2; value SW_PUSH_SMALL -> BOTÓN RESET
- renumbered C9 to C2, C11 to C3, D12 to D1, D11 to D2, D10 to D3, D9 to D4, P1 to P5, R18 to R1, R17 to R2, R16 to R3, R15 to R4, R14 to R7
Connections:
- net labels added: BOTÓN 1, BOTÓN 2
- net labels removed: SWITCH
- wire segments 129 -> 128
Other:
- note removed: "Botones"
- moved on the sheet: P1, P2, R6, SW2

Commit message: Colocados 8 sensores en la placa.
Connections:
- net labels added: SENSOR 7, SENSOR 8
- wire segments 128 -> 132
Changed lines of the file:
@@
 Sheet 1 4
 Title "Tito, el autito más bonito"
-Date "5 jul 2014"
+Date "18 jul 2014"
 Rev "0.3"
 Comp ""
@@
 	1    0    0    -1
 $EndComp
-$Sheet
-S 6500 3150 1250 1350
-U 5391786C
-F0 "Sensores" 50
-F1 "Sensores.sch" 50
-F2 "Habilitador sensores" I L 6500 3450 60
-F3 "Sensor 1" I L 6500 3650 60
-F4 "Sensor 2" I L 6500 3800 60
-F5 "Sensor 3" I L 6500 3950 60
-F6 "Sensor 4" I L 6500 4100 60
-F7 "Sensor 5" I L 6500 4250 60
-F8 "Sensor 6" I L 6500 4400 60
-F9 "Gnd" I R 7750 4250 60
-F10 "+5V" I L 6500 3300 60
-$EndSheet
 $Comp
 L GND #PWR024
@@
 Text Label 8100 6550 0    60   ~ 0
 BOTÓN 2
+$Sheet
+S 6500 3150 1250 1650
+U 5391786C
+F0 "Sensores" 50
+F1 "Sensores.sch" 50
+F2 "Habilitador sensores" I L 6500 3450 60
+F3 "Sensor 1" I L 6500 3650 60
+F4 "Sensor 2" I L 6500 3800 60
+F5 "Sensor 3" I L 6500 3950 60
+F6 "Sensor 4" I L 6500 4100 60
+F7 "Sensor 5" I L 6500 4250 60
+F8 "Sensor 6" I L 6500 4400 60
+F9 "Gnd" I R 7750 4250 60
+F10 "+5V" I L 6500 3300 60
+F11 "Sensor 7" I L 6500 4550 60
+F12 "Sensor 8" I L 6500 4700 60
+$EndSheet
+Text Label 1200 6100 0    60   ~ 0
+SENSOR 7
+Text Label 1200 6200 0    60   ~ 0
+SENSOR 8
+Wire Wire Line
+	1200 6100 1650 6100
+Wire Wire Line
+	1650 6200 1200 6200
+Text Label 6000 4550 0    60   ~ 0
+SENSOR 7
+Text Label 6000 4700 0    60   ~ 0
+SENSOR 8
+Wire Wire Line
+	6500 4550 6000 4550
+Wire Wire Line
+	6500 4700 6000 4700
 $EndSCHEMATC

Commit message: Terminamos de posicionar componentes, y comenzamos el routeo
Parts:
- added P11, P12: ADICIONAL 3,3V, ~, symbol CONN_1
Connections:
- wire segments 132 -> 133
Changed lines of the file:
@@
 Sheet 1 4
 Title "Tito, el autito más bonito"
-Date "16 aug 2014"
+Date "20 aug 2014"
 Rev "0.3"
 Comp ""
@@
 $EndSheet
 $Comp
-L GND #PWR01
+L GND #PWR15
 U 1 1 4DF8B78D
 P 7800 6900
-F 0 "#PWR01" H 7800 6900 30  0001 C CNN
+F 0 "#PWR15" H 7800 6900 30  0001 C CNN
 F 1 "GND" H 7800 6830 30  0001 C CNN
 F 2 "" H 7800 6900 60  0001 C CNN
@@
 $EndComp
 $Comp
-L +5V #PWR02
+L +5V #PWR2
 U 1 1 4DBB5776
 P 1600 4700
-F 0 "#PWR02" H 1600 4790 20  0001 C CNN
+F 0 "#PWR2" H 1600 4790 20  0001 C CNN
 F 1 "+5V" H 1600 4790 30  0000 C CNN
 F 2 "" H 1600 4700 60  0001 C CNN
@@
 MOSI
 $Comp
-L GND #PWR03
+L GND #PWR8
 U 1 1 4DA49E6B
 P 3100 1550
-F 0 "#PWR03" H 3100 1550 30  0001 C CNN
+F 0 "#PWR8" H 3100 1550 30  0001 C CNN
 F 1 "GND" H 3100 1480 30  0001 C CNN
 F 2 "" H 3100 1550 60  0001 C CNN
@@
 $EndComp
 $Comp
-L +5V #PWR04
+L +5V #PWR7
 U 1 1 4DA49E66
 P 3100 1250
-F 0 "#PWR04" H 3100 1340 20  0001 C CNN
+F 0 "#PWR7" H 3100 1340 20  0001 C CNN
 F 1 "+5V" H 3100 1340 30  0000 C CNN
 F 2 "" H 3100 1250 60  0001 C CNN
@@
 MOSI
 $Comp
-L GND #PWR05
+L GND #PWR3
 U 1 1 4DA49DEE
 P 1600 7100
-F 0 "#PWR05" H 1600 7100 30  0001 C CNN
+F 0 "#PWR3" H 1600 7100 30  0001 C CNN
 F 1 "GND" H 1600 7030 30  0001 C CNN
 F 2 "" H 1600 7100 60  0001 C CNN
@@
 $EndComp
 $Comp
-L GND #PWR06
+L GND #PWR27
 U 1 1 50A6D373
 P 10000 6950
-F 0 "#PWR06" H 10000 6950 30  0001 C CNN
+F 0 "#PWR27" H 10000 6950 30  0001 C CNN
 F 1 "GND" H 10000 6880 30  0001 C CNN
 F 2 "" H 10000 6950 60  0001 C CNN
@@
 $EndComp
 $Comp
-L +5V #PWR07
+L +5V #PWR25
 U 1 1 50A6D5B8
 P 9350 6050
-F 0 "#PWR07" H 9350 6140 20  0001 C CNN
+F 0 "#PWR25" H 9350 6140 20  0001 C CNN
 F 1 "+5V" H 9350 6140 30  0000 C CNN
 F 2 "" H 9350 6050 60  0001 C CNN
@@
 $EndComp
 $Comp
-L +5V #PWR08
+L +5V #PWR5
 U 1 1 50CBEEC1
 P 2650 2350
-F 0 "#PWR08" H 2650 2440 20  0001 C CNN
+F 0 "#PWR5" H 2650 2440 20  0001 C CNN
 F 1 "+5V" H 2650 2440 30  0000 C CNN
 F 2 "" H 2650 2350 60  0001 C CNN
@@
 $EndComp
 $Comp
-L +5V #PWR09
+L +5V #PWR14
 U 1 1 50CC0626
 P 7600 5950
-F 0 "#PWR09" H 7600 6040 20  0001 C CNN
+F 0 "#PWR14" H 7600 6040 20  0001 C CNN
 F 1 "+5V" H 7600 6040 30  0000 C CNN
 F 2 "" H 7600 5950 60  0001 C CNN
@@
 LED4
 $Comp
-L GND #PWR010
+L GND #PWR6
 U 1 1 50D4ECDC
 P 2650 2750
-F 0 "#PWR010" H 2650 2750 30  0001 C CNN
+F 0 "#PWR6" H 2650 2750 30  0001 C CNN
 F 1 "GND" H 2650 2680 30  0001 C CNN
 F 2 "" H 2650 2750 60  0001 C CNN
@@
 $EndComp
 $Comp
-L GND #PWR011
+L GND #PWR1
 U 1 1 5127FDB3
 P 1550 5900
-F 0 "#PWR011" H 1550 5900 30  0001 C CNN
+F 0 "#PWR1" H 1550 5900 30  0001 C CNN
 F 1 "GND" H 1550 5830 30  0001 C CNN
 F 2 "" H 1550 5900 60  0001 C CNN
@@
 $EndComp
 $Comp
-L GND #PWR012
+L GND #PWR23
 U 1 1 51280AFC
 P 8750 6900
-F 0 "#PWR012" H 8750 6900 30  0001 C CNN
+F 0 "#PWR23" H 8750 6900 30  0001 C CNN
 F 1 "GND" H 8750 6830 30  0001 C CNN
 F 2 "" H 8750 6900 60  0001 C CNN
@@
 $EndComp
 $Comp
-L +5V #PWR013
+L +5V #PWR22
 U 1 1 51280B0F
 P 8550 5950
-F 0 "#PWR013" H 8550 6040 20  0001 C CNN
+F 0 "#PWR22" H 8550 6040 20  0001 C CNN
 F 1 "+5V" H 8550 6040 30  0000 C CNN
 F 2 "" H 8550 5950 60  0001 C CNN
@@
 $EndComp
 $Comp
-L +3,3V #PWR014
+L +3,3V #PWR9
 U 1 1 52FEAFF7
 P 4550 1950
-F 0 "#PWR014" H 4550 1910 30  0001 C CNN
+F 0 "#PWR9" H 4550 1910 30  0001 C CNN
 F 1 "+3,3V" H 4550 2060 30  0000 C CNN
 F 2 "" H 4550 1950 60  0001 C CNN
@@
 HABILITADOR SENSORES
 $Comp
-L +3,3V #PWR015
+L +3,3V #PWR13
 U 1 1 52FEB95C
 P 7100 4950
-F 0 "#PWR015" H 7100 4910 30  0001 C CNN
+F 0 "#PWR13" H 7100 4910 30  0001 C CNN
 F 1 "+3,3V" H 7100 5060 30  0000 C CNN
 F 2 "" H 7100 4950 60  0001 C CNN
@@
 $EndComp
 $Comp
-L GND #PWR016
+L GND #PWR24
 U 1 1 52FEC00C
 P 9050 4250
-F 0 "#PWR016" H 9050 4250 30  0001 C CNN
+F 0 "#PWR24" H 9050 4250 30  0001 C CNN
 F 1 "GND" H 9050 4180 30  0001 C CNN
 F 2 "" H 9050 4250 60  0001 C CNN
@@
 $EndComp
 $Comp
-L +BATT #PWR017
+L +BATT #PWR18
 U 1 1 5390D35E
 P 8350 1700
-F 0 "#PWR017" H 8350 1650 20  0001 C CNN
+F 0 "#PWR18" H 8350 1650 20  0001 C CNN
 F 1 "+BATT" H 8350 1800 30  0000 C CNN
 F 2 "" H 8350 1700 60  0001 C CNN
@@
 $EndComp
 $Comp
-L +5V #PWR018
+L +5V #PWR20
 U 1 1 5390D39A
 P 8350 2200
-F 0 "#PWR018" H 8350 2290 20  0001 C CNN
+F 0 "#PWR20" H 8350 2290 20  0001 C CNN
 F 1 "+5V" H 8350 2290 30  0000 C CNN
 F 2 "" H 8350 2200 60  0001 C CNN
@@
 $EndComp
 $Comp
-L +3.3V #PWR019
+L +3.3V #PWR21
 U 1 1 5390D3B8
 P 8350 2500
-F 0 "#PWR019" H 8350 2460 30  0001 C CNN
+F 0 "#PWR21" H 8350 2460 30  0001 C CNN
 F 1 "+3.3V" H 8350 2610 30  0000 C CNN
 F 2 "" H 8350 2500 60  0001 C CNN
@@
 $EndComp
 $Comp
-L GND #PWR020
+L GND #PWR26
 U 1 1 5390DC7C
 P 9800 2400
-F 0 "#PWR020" H 9800 2400 30  0001 C CNN
+F 0 "#PWR26" H 9800 2400 30  0001 C CNN
 F 1 "GND" H 9800 2330 30  0001 C CNN
 F 2 "" H 9800 2400 60  0001 C CNN
@@
 $EndComp
 $Comp
-L VDD #PWR021
+L VDD #PWR19
 U 1 1 53910297
 P 8350 1950
-F 0 "#PWR021" H 8350 2050 30  0001 C CNN
+F 0 "#PWR19" H 8350 2050 30  0001 C CNN
 F 1 "VDD" H 8350 2060 30  0000 C CNN
 F 2 "" H 8350 1950 60  0001 C CNN
@@
 IN_1B
 $Comp
-L GND #PWR022
+L GND #PWR16
 U 1 1 53916466
 P 7850 2600
-F 0 "#PWR022" H 7850 2600 30  0001 C CNN
+F 0 "#PWR16" H 7850 2600 30  0001 C CNN
 F 1 "GND" H 7850 2530 30  0001 C CNN
 F 2 "" H 7850 2600 60  0001 C CNN
@@
 $EndComp
 $Comp
-L +BATT #PWR023
+L +BATT #PWR10
 U 1 1 5391651A
 P 6400 1400
-F 0 "#PWR023" H 6400 1350 20  0001 C CNN
+F 0 "#PWR10" H 6400 1350 20  0001 C CNN
 F 1 "+BATT" H 6400 1500 30  0000 C CNN
 F 2 "" H 6400 1400 60  0001 C CNN
@@
 $EndComp
 $Comp
-L GND #PWR024
+L GND #PWR17
 U 1 1 53919AC2
 P 7850 4300
-F 0 "#PWR024" H 7850 4300 30  0001 C CNN
+F 0 "#PWR17" H 7850 4300 30  0001 C CNN
 F 1 "GND" H 7850 4230 30  0001 C CNN
 F 2 "" H 7850 4300 60  0001 C CNN
@@
 $EndComp
 $Comp
-L +5V #PWR025
+L +5V #PWR12
 U 1 1 53919C75
 P 6400 3250
-F 0 "#PWR025" H 6400 3340 20  0001 C CNN
+F 0 "#PWR12" H 6400 3340 20  0001 C CNN
 F 1 "+5V" H 6400 3340 30  0000 C CNN
 F 2 "" H 6400 3250 60  0001 C CNN
@@
 $EndSheet
 $Comp
-L +5V #PWR026
+L +5V #PWR11
 U 1 1 5392E344
 P 6400 2350
-F 0 "#PWR026" H 6400 2440 20  0001 C CNN
+F 0 "#PWR11" H 6400 2440 20  0001 C CNN
 F 1 "+5V" H 6400 2440 30  0000 C CNN
 F 2 "" H 6400 2350 60  0001 C CNN
@@
 Wire Wire Line
 	6500 4700 6000 4700
+Wire Wire Line
+	2300 3550 2600 3550
+Connection ~ 2450 3550
+$Comp
+L CONN_1 P12
+U 1 1 53F4D4F0
+P 2450 3400
+F 0 "P12" H 2530 3400 40  0000 L CNN
+F 1 "ADICIONAL 3,3V" H 2450 3455 30  0000 C CNN
+F 2 "~" H 2450 3400 60  0000 C CNN
+F 3 "~" H 2450 3400 60  0000 C CNN
+	1    2450 3400
+	0    -1   -1   0
+$EndComp
+$Comp
+L CONN_1 P11
+U 1 1 53F4D4F6
+P 2300 3400
+F 0 "P11" H 2380 3400 40  0000 L CNN
+F 1 "ADICIONAL 3,3V" H 2300 3455 30  0000 C CNN
+F 2 "~" H 2300 3400 60  0000 C CNN
+F 3 "~" H 2300 3400 60  0000 C CNN
+	1    2300 3400
+	0    -1   -1   0
+$EndComp
+$Comp
+L +3.3V #PWR4
+U 1 1 53F4E1F1
+P 2600 3550
+F 0 "#PWR4" H 2600 3510 30  0001 C CNN
+F 1 "+3.3V" H 2600 3660 30  0000 C CNN
+F 2 "" H 2600 3550 60  0001 C CNN
+F 3 "" H 2600 3550 60  0001 C CNN
+	1    2600 3550
+	1    0    0    -1
+$EndComp
 $EndSCHEMATC

Commit message: Ruteada placa.
Connections:
- wire segments 133 -> 132
- no-connect marks 0 -> 3
Changed lines of the file:
@@
 Sheet 1 4
 Title "Tito, el autito más bonito"
-Date "20 aug 2014"
+Date "22 aug 2014"
 Rev "0.3"
 Comp ""
@@
 Wire Wire Line
 	7600 6500 7600 6600
-Wire Wire Line
-	3550 4850 3800 4850
 Wire Wire Line
 	3550 4950 3950 4950
@@
 $EndSheet
 $Comp
-L GND #PWR15
+L GND #PWR01
 U 1 1 4DF8B78D
 P 7800 6900
-F 0 "#PWR15" H 7800 6900 30  0001 C CNN
+F 0 "#PWR01" H 7800 6900 30  0001 C CNN
 F 1 "GND" H 7800 6830 30  0001 C CNN
 F 2 "" H 7800 6900 60  0001 C CNN
@@
 $EndComp
 $Comp
-L +5V #PWR2
+L +5V #PWR02
 U 1 1 4DBB5776
 P 1600 4700
-F 0 "#PWR2" H 1600 4790 20  0001 C CNN
+F 0 "#PWR02" H 1600 4790 20  0001 C CNN
 F 1 "+5V" H 1600 4790 30  0000 C CNN
 F 2 "" H 1600 4700 60  0001 C CNN
@@
 MOSI
 $Comp
-L GND #PWR8
+L GND #PWR03
 U 1 1 4DA49E6B
 P 3100 1550
-F 0 "#PWR8" H 3100 1550 30  0001 C CNN
+F 0 "#PWR03" H 3100 1550 30  0001 C CNN
 F 1 "GND" H 3100 1480 30  0001 C CNN
 F 2 "" H 3100 1550 60  0001 C CNN
@@
 $EndComp
 $Comp
-L +5V #PWR7
+L +5V #PWR04
 U 1 1 4DA49E66
 P 3100 1250
-F 0 "#PWR7" H 3100 1340 20  0001 C CNN
+F 0 "#PWR04" H 3100 1340 20  0001 C CNN
 F 1 "+5V" H 3100 1340 30  0000 C CNN
 F 2 "" H 3100 1250 60  0001 C CNN
@@
 MOSI
 $Comp
-L GND #PWR3
+L GND #PWR05
 U 1 1 4DA49DEE
 P 1600 7100
-F 0 "#PWR3" H 1600 7100 30  0001 C CNN
+F 0 "#PWR05" H 1600 7100 30  0001 C CNN
 F 1 "GND" H 1600 7030 30  0001 C CNN
 F 2 "" H 1600 7100 60  0001 C CNN
@@
 $EndComp
 $Comp
-L GND #PWR27
+L GND #PWR06
 U 1 1 50A6D373
 P 10000 6950
-F 0 "#PWR27" H 10000 6950 30  0001 C CNN
+F 0 "#PWR06" H 10000 6950 30  0001 C CNN
 F 1 "GND" H 10000 6880 30  0001 C CNN
 F 2 "" H 10000 6950 60  0001 C CNN
@@
 $EndComp
 $Comp
-L +5V #PWR25
+L +5V #PWR07
 U 1 1 50A6D5B8
 P 9350 6050
-F 0 "#PWR25" H 9350 6140 20  0001 C CNN
+F 0 "#PWR07" H 9350 6140 20  0001 C CNN
 F 1 "+5V" H 9350 6140 30  0000 C CNN
 F 2 "" H 9350 6050 60  0001 C CNN
@@
 $EndComp
 $Comp
-L +5V #PWR5
+L +5V #PWR08
 U 1 1 50CBEEC1
 P 2650 2350
-F 0 "#PWR5" H 2650 2440 20  0001 C CNN
+F 0 "#PWR08" H 2650 2440 20  0001 C CNN
 F 1 "+5V" H 2650 2440 30  0000 C CNN
 F 2 "" H 2650 2350 60  0001 C CNN
@@
 $EndComp
 $Comp
-L +5V #PWR14
+L +5V #PWR09
 U 1 1 50CC0626
 P 7600 5950
-F 0 "#PWR14" H 7600 6040 20  0001 C CNN
+F 0 "#PWR09" H 7600 6040 20  0001 C CNN
 F 1 "+5V" H 7600 6040 30  0000 C CNN
 F 2 "" H 7600 5950 60  0001 C CNN
@@
 	1    0    0    -1
 $EndComp
+Text Label 1200 6100 0    60   ~ 0
+SENSOR 1
+Text Label 1200 6200 0    60   ~ 0
+SENSOR 2
 Text Label 4000 5600 2    60   ~ 0
-SENSOR 1
+SENSOR 3
 Text Label 4000 5700 2    60   ~ 0
-SENSOR 2
+SENSOR 4
 Text Label 4000 5800 2    60   ~ 0
-SENSOR 3
+SENSOR 5
 Text Label 4000 5900 2    60   ~ 0
-SENSOR 4
-Text Label 4000 6000 2    60   ~ 0
-SENSOR 5
-Text Label 4000 6100 2    60   ~ 0
 SENSOR 6
 Text Label 3750 4750 2    60   ~ 0
@@
 LED4
 $Comp
-L GND #PWR6
+L GND #PWR010
 U 1 1 50D4ECDC
 P 2650 2750
-F 0 "#PWR6" H 2650 2750 30  0001 C CNN
+F 0 "#PWR010" H 2650 2750 30  0001 C CNN
 F 1 "GND" H 2650 2680 30  0001 C CNN
 F 2 "" H 2650 2750 60  0001 C CNN
@@
 $EndComp
 $Comp
-L GND #PWR1
+L GND #PWR011
 U 1 1 5127FDB3
 P 1550 5900
-F 0 "#PWR1" H 1550 5900 30  0001 C CNN
+F 0 "#PWR011" H 1550 5900 30  0001 C CNN
 F 1 "GND" H 1550 5830 30  0001 C CNN
 F 2 "" H 1550 5900 60  0001 C CNN
@@
 $EndComp
 $Comp
-L GND #PWR23
+L GND #PWR012
 U 1 1 51280AFC
 P 8750 6900
-F 0 "#PWR23" H 8750 6900 30  0001 C CNN
+F 0 "#PWR012" H 8750 6900 30  0001 C CNN
 F 1 "GND" H 8750 6830 30  0001 C CNN
 F 2 "" H 8750 6900 60  0001 C CNN
@@
 $EndComp
 $Comp
-L +5V #PWR22
+L +5V #PWR013
 U 1 1 51280B0F
 P 8550 5950
-F 0 "#PWR22" H 8550 6040 20  0001 C CNN
+F 0 "#PWR013" H 8550 6040 20  0001 C CNN
 F 1 "+5V" H 8550 6040 30  0000 C CNN
 F 2 "" H 8550 5950 60  0001 C CNN
@@
 $EndComp
 $Comp
-L +3,3V #PWR9
+L +3,3V #PWR014
 U 1 1 52FEAFF7
 P 4550 1950
-F 0 "#PWR9" H 4550 1910 30  0001 C CNN
+F 0 "#PWR014" H 4550 1910 30  0001 C CNN
 F 1 "+3,3V" H 4550 2060 30  0000 C CNN
 F 2 "" H 4550 1950 60  0001 C CNN
@@
 HABILITADOR SENSORES
 $Comp
-L +3,3V #PWR13
+L +3,3V #PWR015
 U 1 1 52FEB95C
 P 7100 4950
-F 0 "#PWR13" H 7100 4910 30  0001 C CNN
+F 0 "#PWR015" H 7100 4910 30  0001 C CNN
 F 1 "+3,3V" H 7100 5060 30  0000 C CNN
 F 2 "" H 7100 4950 60  0001 C CNN
@@
 $EndComp
 $Comp
-L GND #PWR24
+L GND #PWR016
 U 1 1 52FEC00C
 P 9050 4250
-F 0 "#PWR24" H 9050 4250 30  0001 C CNN
+F 0 "#PWR016" H 9050 4250 30  0001 C CNN
 F 1 "GND" H 9050 4180 30  0001 C CNN
 F 2 "" H 9050 4250 60  0001 C CNN
@@
 $EndComp
 $Comp
-L +BATT #PWR18
+L +BATT #PWR017
 U 1 1 5390D35E
 P 8350 1700
-F 0 "#PWR18" H 8350 1650 20  0001 C CNN
+F 0 "#PWR017" H 8350 1650 20  0001 C CNN
 F 1 "+BATT" H 8350 1800 30  0000 C CNN
 F 2 "" H 8350 1700 60  0001 C CNN
@@
 $EndComp
 $Comp
-L +5V #PWR20
+L +5V #PWR018
 U 1 1 5390D39A
 P 8350 2200
-F 0 "#PWR20" H 8350 2290 20  0001 C CNN
+F 0 "#PWR018" H 8350 2290 20  0001 C CNN
 F 1 "+5V" H 8350 2290 30  0000 C CNN
 F 2 "" H 8350 2200 60  0001 C CNN
@@
 $EndComp
 $Comp
-L +3.3V #PWR21
+L +3.3V #PWR019
 U 1 1 5390D3B8
 P 8350 2500
-F 0 "#PWR21" H 8350 2460 30  0001 C CNN
+F 0 "#PWR019" H 8350 2460 30  0001 C CNN
 F 1 "+3.3V" H 8350 2610 30  0000 C CNN
 F 2 "" H 8350 2500 60  0001 C CNN
@@
 $EndComp
 $Comp
-L GND #PWR26
+L GND #PWR020
 U 1 1 5390DC7C
 P 9800 2400
-F 0 "#PWR26" H 9800 2400 30  0001 C CNN
+F 0 "#PWR020" H 9800 2400 30  0001 C CNN
 F 1 "GND" H 9800 2330 30  0001 C CNN
 F 2 "" H 9800 2400 60  0001 C CNN
@@
 $EndComp
 $Comp
-L VDD #PWR19
+L VDD #PWR021
 U 1 1 53910297
 P 8350 1950
-F 0 "#PWR19" H 8350 2050 30  0001 C CNN
+F 0 "#PWR021" H 8350 2050 30  0001 C CNN
 F 1 "VDD" H 8350 2060 30  0000 C CNN
 F 2 "" H 8350 1950 60  0001 C CNN
@@
 IN_1B
 $Comp
-L GND #PWR16
+L GND #PWR022
 U 1 1 53916466
 P 7850 2600
-F 0 "#PWR16" H 7850 2600 30  0001 C CNN
+F 0 "#PWR022" H 7850 2600 30  0001 C CNN
 F 1 "GND" H 7850 2530 30  0001 C CNN
 F 2 "" H 7850 2600 60  0001 C CNN
@@
 $EndComp
 $Comp
-L +BATT #PWR10
+L +BATT #PWR023
 U 1 1 5391651A
 P 6400 1400
-F 0 "#PWR10" H 6400 1350 20  0001 C CNN
+F 0 "#PWR023" H 6400 1350 20  0001 C CNN
 F 1 "+BATT" H 6400 1500 30  0000 C CNN
 F 2 "" H 6400 1400 60  0001 C CNN
@@
 $EndComp
 $Comp
-L GND #PWR17
+L GND #PWR024
 U 1 1 53919AC2
 P 7850 4300
-F 0 "#PWR17" H 7850 4300 30  0001 C CNN
+F 0 "#PWR024" H 7850 4300 30  0001 C CNN
 F 1 "GND" H 7850 4230 30  0001 C CNN
 F 2 "" H 7850 4300 60  0001 C CNN
@@
 $EndComp
 $Comp
-L +5V #PWR12
+L +5V #PWR025
 U 1 1 53919C75
 P 6400 3250
-F 0 "#PWR12" H 6400 3340 20  0001 C CNN
+F 0 "#PWR025" H 6400 3340 20  0001 C CNN
 F 1 "+5V" H 6400 3340 30  0000 C CNN
 F 2 "" H 6400 3250 60  0001 C CNN
@@
 $EndSheet
 $Comp
-L +5V #PWR11
+L +5V #PWR026
 U 1 1 5392E344
 P 6400 2350
-F 0 "#PWR11" H 6400 2440 20  0001 C CNN
+F 0 "#PWR026" H 6400 2440 20  0001 C CNN
 F 1 "+5V" H 6400 2440 30  0000 C CNN
 F 2 "" H 6400 2350 60  0001 C CNN
@@
 Text Label 6200 2550 0    60   ~ 0
 SERVO
-Text Label 3800 4850 2    60   ~ 0
+Text Label 3950 4600 2    60   ~ 0
 SERVO
 $Comp
@@
 F12 "Sensor 8" I L 6500 4700 60
 $EndSheet
-Text Label 1200 6100 0    60   ~ 0
+Text Label 4000 6000 2    60   ~ 0
 SENSOR 7
-Text Label 1200 6200 0    60   ~ 0
+Text Label 4000 6100 2    60   ~ 0
 SENSOR 8
 Wire Wire Line
@@
 $EndComp
 $Comp
-L +3.3V #PWR4
+L +3.3V #PWR027
 U 1 1 53F4E1F1
 P 2600 3550
-F 0 "#PWR4" H 2600 3510 30  0001 C CNN
+F 0 "#PWR027" H 2600 3510 30  0001 C CNN
 F 1 "+3.3V" H 2600 3660 30  0000 C CNN
 F 2 "" H 2600 3550 60  0001 C CNN
@@
 	1    0    0    -1
 $EndComp
+NoConn ~ 3950 4600
+NoConn ~ 3550 4850
+NoConn ~ 6200 2550
 $EndSCHEMATC
