File: Placas/Placa_Tito_2013/Placa_principal/Alimentacion.sch (KiCad schematic (older format))
At the start: 12 parts

Commit message: Ajustes de estandarización de nombres en componentes y etiquetas del esquemático. Removido cny70 del .pro, agregado datasheet tcrt1000
Parts:
- C? (x2): value 10 nF -> 10 n
- C? (x2): value 220 uF -> 220 u
- C? (x2): value 100 nF -> 100 n
- P?: value Bateria 7,2V -> Batería 7,2V
- P?: value Bateria 3,6V -> Batería 3,6V
Connections:
- net labels added: +Batt, Gnd, Vdd
- net labels removed: +BATT
- wire segments 52 -> 57

Commit message: Terminado esquemático. Comenzado a asociar componentes.
Parts:
- removed SW? (x2): DUAL_SWITCH_INV, symbol DUAL_SWITCH_INV
- added SW4: INTERRUPTOR BATERÍA 7,2V, ~, symbol SWITCH_INV
- added SW5: INTERRUPTOR BATERÍA 3,7V, ~, symbol SWITCH_INV
- gave numbers to parts that had none: 10
Changed lines of the file:
@@
-EESchema Schematic File Version 2  date jue 12 jun 2014 20:15:01 ART
+EESchema Schematic File Version 2
 LIBS:power
 LIBS:device
@@
 LIBS:drv8833
 LIBS:placa_principal-cache
-EELAYER 25  0
+EELAYER 27 0
 EELAYER END
-$Descr A4 11700 8267
+$Descr A4 11693 8268
 encoding utf-8
 Sheet 4 4
 Title ""
-Date "12 jun 2014"
+Date "14 jun 2014"
 Rev ""
 Comp ""
@@
 GND
 $Comp
-L C C?
+L C C14
 U 1 1 5390D675
 P 6950 3350
-F 0 "C?" H 7000 3450 50  0000 L CNN
+F 0 "C14" H 7000 3450 50  0000 L CNN
 F 1 "10 n" H 7000 3250 50  0000 L CNN
+F 2 "" H 6950 3350 60  0001 C CNN
+F 3 "" H 6950 3350 60  0001 C CNN
 	1    6950 3350
 	1    0    0    -1
 $EndComp
 $Comp
-L REG_104-5 U?
+L REG_104-5 U8
 U 1 1 5390D681
 P 6150 3150
-F 0 "U?" H 5900 3350 60  0000 C CNN
+F 0 "U8" H 5900 3350 60  0000 C CNN
 F 1 "REG_104-5" H 6150 3450 60  0000 C CNN
+F 2 "" H 6150 3150 60  0001 C CNN
+F 3 "" H 6150 3150 60  0001 C CNN
 	1    6150 3150
 	1    0    0    -1
 $EndComp
 $Comp
-L CONN_2 P?
+L CONN_2 P9
 U 1 1 5390D68D
 P 3400 3150
-F 0 "P?" V 3350 3150 40  0000 C CNN
+F 0 "P9" V 3350 3150 40  0000 C CNN
 F 1 "Batería 7,2V" V 3450 3150 40  0000 C CNN
+F 2 "" H 3400 3150 60  0001 C CNN
+F 3 "" H 3400 3150 60  0001 C CNN
 	1    3400 3150
 	-1   0    0    1
 $EndComp
 $Comp
-L CAPAPOL C?
+L CAPAPOL C12
 U 1 1 5390D693
 P 5500 3500
-F 0 "C?" H 5550 3600 50  0000 L CNN
+F 0 "C12" H 5550 3600 50  0000 L CNN
 F 1 "220 u" H 5550 3400 50  0000 L CNN
+F 2 "" H 5500 3500 60  0001 C CNN
+F 3 "" H 5500 3500 60  0001 C CNN
 	1    5500 3500
 	1    0    0    -1
 $EndComp
 $Comp
-L CONN_2 P?
+L CONN_2 P10
 U 1 1 5390D699
 P 4900 2200
-F 0 "P?" V 4850 2200 40  0000 C CNN
+F 0 "P10" V 4850 2200 40  0000 C CNN
 F 1 "Batería 3,6V" V 4950 2200 40  0000 C CNN
+F 2 "" H 4900 2200 60  0001 C CNN
+F 3 "" H 4900 2200 60  0001 C CNN
 	1    4900 2200
 	-1   0    0    1
 $EndComp
 $Comp
-L C C?
+L C C15
 U 1 1 5390D6CB
 P 6950 5100
-F 0 "C?" H 7000 5200 50  0000 L CNN
+F 0 "C15" H 7000 5200 50  0000 L CNN
 F 1 "10 n" H 7000 5000 50  0000 L CNN
+F 2 "" H 6950 5100 60  0001 C CNN
+F 3 "" H 6950 5100 60  0001 C CNN
 	1    6950 5100
 	1    0    0    -1
 $EndComp
 $Comp
-L REG_104-5 U?
+L REG_104-5 U9
 U 1 1 5390D6D1
 P 6150 4900
-F 0 "U?" H 5900 5100 60  0000 C CNN
+F 0 "U9" H 5900 5100 60  0000 C CNN
 F 1 "REG_104-3.3" H 6150 5200 60  0000 C CNN
+F 2 "" H 6150 4900 60  0001 C CNN
+F 3 "" H 6150 4900 60  0001 C CNN
 	1    6150 4900
 	1    0    0    -1
 $EndComp
 $Comp
-L CAPAPOL C?
+L CAPAPOL C13
 U 1 1 5390D6DD
 P 5500 5250
-F 0 "C?" H 5550 5350 50  0000 L CNN
+F 0 "C13" H 5550 5350 50  0000 L CNN
 F 1 "220 u" H 5550 5150 50  0000 L CNN
+F 2 "" H 5500 5250 60  0001 C CNN
+F 3 "" H 5500 5250 60  0001 C CNN
 	1    5500 5250
 	1    0    0    -1
 $EndComp
 $Comp
-L DUAL_SWITCH_INV SW?
-U 1 1 5390D6F5
-P 4400 3300
-F 0 "SW?" H 4200 3450 50  0000 C CNN
-F 1 "DUAL_SWITCH_INV" H 4250 3150 50  0000 C CNN
-	1    4400 3300
-	-1   0    0    1
-$EndComp
-$Comp
-L DUAL_SWITCH_INV SW?
-U 1 1 5390D6FB
-P 4400 5150
-F 0 "SW?" H 4200 5300 50  0000 C CNN
-F 1 "DUAL_SWITCH_INV" H 4250 5000 50  0000 C CNN
-	1    4400 5150
-	-1   0    0    1
-$EndComp
-$Comp
-L C C?
+L C C10
 U 1 1 5390D8D2
 P 5150 3500
-F 0 "C?" H 5150 3600 40  0000 L CNN
+F 0 "C10" H 5150 3600 40  0000 L CNN
 F 1 "100 n" H 5156 3415 40  0000 L CNN
 F 2 "~" H 5188 3350 30  0000 C CNN
@@
 $EndComp
 $Comp
-L C C?
+L C C11
 U 1 1 5390DAD4
 P 5150 5250
-F 0 "C?" H 5150 5350 40  0000 L CNN
+F 0 "C11" H 5150 5350 40  0000 L CNN
 F 1 "100 n" H 5156 5165 40  0000 L CNN
 F 2 "~" H 5188 5100 30  0000 C CNN
@@
 Text HLabel 5550 4950 0    60   Input ~ 0
 +3,3V
+$Comp
+L SWITCH_INV SW4
+U 1 1 539C41D8
+P 4400 3300
+F 0 "SW4" H 4200 3450 50  0000 C CNN
+F 1 "INTERRUPTOR BATERÍA 7,2V" H 4250 3150 50  0000 C CNN
+F 2 "~" H 4400 3300 60  0000 C CNN
+F 3 "~" H 4400 3300 60  0000 C CNN
+	1    4400 3300
+	-1   0    0    1
+$EndComp
+$Comp
+L SWITCH_INV SW5
+U 1 1 539C41EF
+P 4400 5150
+F 0 "SW5" H 4200 5300 50  0000 C CNN
+F 1 "INTERRUPTOR BATERÍA 3,7V" H 4250 5000 50  0000 C CNN
+F 2 "~" H 4400 5150 60  0000 C CNN
+F 3 "~" H 4400 5150 60  0000 C CNN
+	1    4400 5150
+	-1   0    0    1
+$EndComp
 $EndSCHEMATC

Commit message: Colocados 8 sensores en la placa.
Parts:
- renumbered U8 to U10, U9 to U11
Changed lines of the file:
@@
 Sheet 4 4
 Title ""
-Date "5 jul 2014"
+Date "18 jul 2014"
 Rev ""
 Comp ""
@@
 $EndComp
 $Comp
-L REG_104-5 U8
+L REG_104-5 U10
 U 1 1 5390D681
 P 6150 3150
-F 0 "U8" H 5900 3350 60  0000 C CNN
+F 0 "U10" H 5900 3350 60  0000 C CNN
 F 1 "REG_104-5" H 6150 3450 60  0000 C CNN
 F 2 "" H 6150 3150 60  0001 C CNN
@@
 $EndComp
 $Comp
-L REG_104-5 U9
+L REG_104-5 U11
 U 1 1 5390D6D1
 P 6150 4900
-F 0 "U9" H 5900 5100 60  0000 C CNN
+F 0 "U11" H 5900 5100 60  0000 C CNN
 F 1 "REG_104-3.3" H 6150 5200 60  0000 C CNN
 F 2 "" H 6150 4900 60  0001 C CNN

Commit message: Empezados a colocar componentes en la placa
Parts:
- SW5: value INTERRUPTOR BATERÍA 3,7V -> INTERRUPTOR REGULADOR 3,3V
Changed lines of the file:
@@
 Sheet 4 4
 Title ""
-Date "18 jul 2014"
+Date "1 aug 2014"
 Rev ""
 Comp ""
@@
 P 4400 5150
 F 0 "SW5" H 4200 5300 50  0000 C CNN
-F 1 "INTERRUPTOR BATERÍA 3,7V" H 4250 5000 50  0000 C CNN
+F 1 "INTERRUPTOR REGULADOR 3,3V" H 4250 5000 50  0000 C CNN
 F 2 "~" H 4400 5150 60  0000 C CNN
 F 3 "~" H 4400 5150 60  0000 C CNN

Commit message: Seguimos posicionando componentes en el PBC
Changed lines of the file:
@@
 $Descr A4 11693 8268
 encoding utf-8
-Sheet 4 4
+Sheet 3 4
 Title ""
-Date "1 aug 2014"
+Date "16 aug 2014"
 Rev ""
 Comp ""
@@
 	-1   0    0    1
 $EndComp
+Connection ~ 5150 4800
 $EndSCHEMATC
