File: Placas/Placa_Tito_2013/Placa_principal/Control_motores.sch (KiCad schematic (older format))
At the start: 10 parts

Commit message: Ajustes de estandarización de nombres en componentes y etiquetas del esquemático. Removido cny70 del .pro, agregado datasheet tcrt1000
Parts:
- C? (x2): value 10 nF -> 10 n
- C?: value 2,2 uF -> 2,2 u
- C?: value 2200 uF -> 2200 u
- C?: value 100uF -> 100 u
- R?: value R -> 47 k
Connections:
- net labels added: +Batt, ALIMENTACIÓN, Alimentación Servo, Gnd, MOTOR A SALIDA 1, MOTOR A SALIDA 2, MOTOR B SALIDA 1, MOTOR B SALIDA 2, SERVO
- net labels removed: +BATT, Alimentacion, Alimentacion Servo, Motor A salida 1, Motor A salida 2, Motor B salida 1, Motor B salida 2, servo
- wire segments 47 -> 53
- no-connect marks 0 -> 1

Commit message: Terminado esquemático. Comenzado a asociar componentes.
Parts:
- gave numbers to parts that had none: 10
Changed lines of the file:
@@
-EESchema Schematic File Version 2  date jue 12 jun 2014 20:15:01 ART
+EESchema Schematic File Version 2
 LIBS:power
 LIBS:device
@@
 LIBS:drv8833
 LIBS:placa_principal-cache
-EELAYER 25  0
+EELAYER 27 0
 EELAYER END
-$Descr A4 11700 8267
+$Descr A4 11693 8268
 encoding utf-8
 Sheet 2 4
 Title ""
-Date "12 jun 2014"
+Date "14 jun 2014"
 Rev ""
 Comp ""
@@
 GND
 $Comp
-L DRV8833 U?
+L DRV8833 U1
 U 1 1 53910CF9
 P 5050 3200
-F 0 "U?" H 5100 3550 60  0000 C CNN
+F 0 "U1" H 5100 3550 60  0000 C CNN
 F 1 "DRV8833" H 5050 3650 60  0000 C CNN
 F 2 "~" H 5050 3200 60  0000 C CNN
@@
 $EndComp
 $Comp
-L R R?
+L R R8
 U 1 1 53910D0B
 P 4100 2550
-F 0 "R?" V 4180 2550 40  0000 C CNN
+F 0 "R8" V 4180 2550 40  0000 C CNN
 F 1 "47 k" V 4107 2551 40  0000 C CNN
 F 2 "~" V 4030 2550 30  0000 C CNN
@@
 $EndComp
 $Comp
-L C C?
+L C C5
 U 1 1 53910D3D
 P 7000 3500
-F 0 "C?" H 7000 3600 40  0000 L CNN
+F 0 "C5" H 7000 3600 40  0000 L CNN
 F 1 "10 n" H 7006 3415 40  0000 L CNN
 F 2 "~" H 7038 3350 30  0000 C CNN
@@
 $EndComp
 $Comp
-L CAPAPOL C?
+L CAPAPOL C8
 U 1 1 53910D48
 P 8000 3300
-F 0 "C?" H 8050 3400 40  0000 L CNN
+F 0 "C8" H 8050 3400 40  0000 L CNN
 F 1 "2,2 u" H 8050 3200 40  0000 L CNN
 F 2 "~" H 8100 3150 30  0000 C CNN
@@
 $EndComp
 $Comp
-L CAPAPOL C?
+L CAPAPOL C6
 U 1 1 53910D57
 P 7300 3500
-F 0 "C?" H 7350 3600 40  0000 L CNN
+F 0 "C6" H 7350 3600 40  0000 L CNN
 F 1 "2200 u" H 7350 3400 40  0000 L CNN
 F 2 "~" H 7400 3350 30  0000 C CNN
@@
 $EndComp
 $Comp
-L C C?
+L C C7
 U 1 1 53910D67
 P 7700 3500
-F 0 "C?" H 7700 3600 40  0000 L CNN
+F 0 "C7" H 7700 3600 40  0000 L CNN
 F 1 "10 n" H 7706 3415 40  0000 L CNN
 F 2 "~" H 7738 3350 30  0000 C CNN
@@
 Motor B Entrada 1
 $Comp
-L CONN_2 P?
+L CONN_2 P8
 U 1 1 5391385D
 P 6000 2150
-F 0 "P?" V 5950 2150 40  0000 C CNN
+F 0 "P8" V 5950 2150 40  0000 C CNN
 F 1 "Motor 2" V 6050 2150 40  0000 C CNN
+F 2 "" H 6000 2150 60  0001 C CNN
+F 3 "" H 6000 2150 60  0001 C CNN
 	1    6000 2150
 	-1   0    0    -1
 $EndComp
 $Comp
-L CONN_2 P?
+L CONN_2 P7
 U 1 1 53913863
 P 6000 1700
-F 0 "P?" V 5950 1700 40  0000 C CNN
+F 0 "P7" V 5950 1700 40  0000 C CNN
 F 1 "Motor 1" V 6050 1700 40  0000 C CNN
+F 2 "" H 6000 1700 60  0001 C CNN
+F 3 "" H 6000 1700 60  0001 C CNN
 	1    6000 1700
 	-1   0    0    -1
@@
 ALIMENTACIÓN
 $Comp
-L CONN_3 K?
+L CONN_3 K1
 U 1 1 5392D7E5
 P 8250 1900
-F 0 "K?" V 8200 1900 50  0000 C CNN
+F 0 "K1" V 8200 1900 50  0000 C CNN
 F 1 "Servo" V 8300 1900 40  0000 C CNN
+F 2 "" H 8250 1900 60  0001 C CNN
+F 3 "" H 8250 1900 60  0001 C CNN
 	1    8250 1900
 	-1   0    0    1
 $EndComp
 $Comp
-L CAPAPOL C?
+L CAPAPOL C9
 U 1 1 5392D7F2
 P 9100 1900
-F 0 "C?" H 9150 2000 50  0000 L CNN
+F 0 "C9" H 9150 2000 50  0000 L CNN
 F 1 "100 u" H 9150 1800 50  0000 L CNN
+F 2 "" H 9100 1900 60  0001 C CNN
+F 3 "" H 9100 1900 60  0001 C CNN
 	1    9100 1900
 	1    0    0    -1
