File: Placas/Placa_Tito_2013/Placa_principal/Sensores.sch (KiCad schematic (older format))
At the start: 24 parts

Commit message: Ajustes de estandarización de nombres en componentes y etiquetas del esquemático. Removido cny70 del .pro, agregado datasheet tcrt1000
Parts:
- R? (x6): value R sensor -> 180
- RV? (x6): value POT -> POT 20 k
Connections:
- net labels added: Gnd
- wire segments 81 -> 94
Other:
- moved on the sheet: R?

Commit message: Terminado esquemático. Comenzado a asociar componentes.
Parts:
- gave numbers to parts that had none: 24
Changed lines of the file:
@@
-EESchema Schematic File Version 2  date jue 12 jun 2014 20:15:01 ART
+EESchema Schematic File Version 2
 LIBS:power
 LIBS:device
@@
 LIBS:drv8833
 LIBS:placa_principal-cache
-EELAYER 25  0
+EELAYER 27 0
 EELAYER END
-$Descr A4 11700 8267
+$Descr A4 11693 8268
 encoding utf-8
 Sheet 3 4
 Title ""
-Date "12 jun 2014"
+Date "14 jun 2014"
 Rev ""
 Comp ""
@@
 GND
 $Comp
-L POT RV?
+L POT RV3
 U 1 1 53917AA3
 P 7100 3000
-F 0 "RV?" H 7100 2900 50  0000 C CNN
+F 0 "RV3" H 7100 2900 50  0000 C CNN
 F 1 "POT 20 k" H 7100 3000 50  0000 C CNN
+F 2 "" H 7100 3000 60  0001 C CNN
+F 3 "" H 7100 3000 60  0001 C CNN
 	1    7100 3000
 	1    0    0    -1
 $EndComp
 $Comp
-L POT RV?
+L POT RV1
 U 1 1 53917AA9
 P 7100 2400
-F 0 "RV?" H 7100 2300 50  0000 C CNN
+F 0 "RV1" H 7100 2300 50  0000 C CNN
 F 1 "POT 20 k" H 7100 2400 50  0000 C CNN
+F 2 "" H 7100 2400 60  0001 C CNN
+F 3 "" H 7100 2400 60  0001 C CNN
 	1    7100 2400
 	1    0    0    -1
 $EndComp
 $Comp
-L POT RV?
+L POT RV4
 U 1 1 53917AAF
 P 7100 3300
-F 0 "RV?" H 7100 3200 50  0000 C CNN
+F 0 "RV4" H 7100 3200 50  0000 C CNN
 F 1 "POT 20 k" H 7100 3300 50  0000 C CNN
+F 2 "" H 7100 3300 60  0001 C CNN
+F 3 "" H 7100 3300 60  0001 C CNN
 	1    7100 3300
 	1    0    0    -1
 $EndComp
 $Comp
-L POT RV?
+L POT RV2
 U 1 1 53917AB5
 P 7100 2700
-F 0 "RV?" H 7100 2600 50  0000 C CNN
+F 0 "RV2" H 7100 2600 50  0000 C CNN
 F 1 "POT 20 k" H 7100 2700 50  0000 C CNN
+F 2 "" H 7100 2700 60  0001 C CNN
+F 3 "" H 7100 2700 60  0001 C CNN
 	1    7100 2700
 	1    0    0    -1
@@
 SENSOR 4
 $Comp
-L R R?
+L R R18
 U 1 1 53917ABC
 P 6550 3300
-F 0 "R?" V 6630 3300 50  0000 C CNN
+F 0 "R18" V 6630 3300 50  0000 C CNN
 F 1 "100" V 6550 3300 50  0000 C CNN
+F 2 "" H 6550 3300 60  0001 C CNN
+F 3 "" H 6550 3300 60  0001 C CNN
 	1    6550 3300
 	0    1    1    0
@@
 Resistencias\nde seguridad
 $Comp
-L R R?
+L R R17
 U 1 1 53917AC3
 P 6550 3000
-F 0 "R?" V 6630 3000 50  0000 C CNN
+F 0 "R17" V 6630 3000 50  0000 C CNN
 F 1 "100" V 6550 3000 50  0000 C CNN
+F 2 "" H 6550 3000 60  0001 C CNN
+F 3 "" H 6550 3000 60  0001 C CNN
 	1    6550 3000
 	0    1    1    0
 $EndComp
 $Comp
-L R R?
+L R R16
 U 1 1 53917AC9
 P 6550 2700
-F 0 "R?" V 6630 2700 50  0000 C CNN
+F 0 "R16" V 6630 2700 50  0000 C CNN
 F 1 "100" V 6550 2700 50  0000 C CNN
+F 2 "" H 6550 2700 60  0001 C CNN
+F 3 "" H 6550 2700 60  0001 C CNN
 	1    6550 2700
 	0    1    1    0
 $EndComp
 $Comp
-L R R?
+L R R15
 U 1 1 53917ACF
 P 6550 2400
-F 0 "R?" V 6630 2400 50  0000 C CNN
+F 0 "R15" V 6630 2400 50  0000 C CNN
 F 1 "100" V 6550 2400 50  0000 C CNN
+F 2 "" H 6550 2400 60  0001 C CNN
+F 3 "" H 6550 2400 60  0001 C CNN
 	1    6550 2400
 	0    1    1    0
@@
 SENSOR 3
 $Comp
-L POT RV?
+L POT RV5
 U 1 1 53917AD6
 P 7100 3600
-F 0 "RV?" H 7100 3500 50  0000 C CNN
+F 0 "RV5" H 7100 3500 50  0000 C CNN
 F 1 "POT 20 k" H 7100 3600 50  0000 C CNN
+F 2 "" H 7100 3600 60  0001 C CNN
+F 3 "" H 7100 3600 60  0001 C CNN
 	1    7100 3600
 	1    0    0    -1
 $EndComp
 $Comp
-L POT RV?
+L POT RV6
 U 1 1 53917ADC
 P 7100 3900
-F 0 "RV?" H 7100 3800 50  0000 C CNN
+F 0 "RV6" H 7100 3800 50  0000 C CNN
 F 1 "POT 20 k" H 7100 3900 50  0000 C CNN
+F 2 "" H 7100 3900 60  0001 C CNN
+F 3 "" H 7100 3900 60  0001 C CNN
 	1    7100 3900
 	1    0    0    -1
@@
 SENSOR 6
 $Comp
-L R R?
+L R R20
 U 1 1 53917AE3
 P 6550 3900
-F 0 "R?" V 6630 3900 50  0000 C CNN
+F 0 "R20" V 6630 3900 50  0000 C CNN
 F 1 "100" V 6550 3900 50  0000 C CNN
+F 2 "" H 6550 3900 60  0001 C CNN
+F 3 "" H 6550 3900 60  0001 C CNN
 	1    6550 3900
 	0    1    1    0
 $EndComp
 $Comp
-L R R?
+L R R19
 U 1 1 53917AEF
 P 6550 3600
-F 0 "R?" V 6630 3600 50  0000 C CNN
+F 0 "R19" V 6630 3600 50  0000 C CNN
 F 1 "100" V 6550 3600 50  0000 C CNN
+F 2 "" H 6550 3600 60  0001 C CNN
+F 3 "" H 6550 3600 60  0001 C CNN
 	1    6550 3600
 	0    1    1    0
@@
 SENSOR 2
 $Comp
-L TCRT1000 U?
+L TCRT1000 U2
 U 1 1 539180FB
 P 3200 2400
-F 0 "U?" H 3200 2400 60  0000 C CNN
+F 0 "U2" H 3200 2400 60  0000 C CNN
 F 1 "TCRT1000" H 3450 2600 60  0000 C CNN
 F 2 "TCRT1000" H 2950 2600 60  0000 C CNN
+F 3 "" H 3200 2400 60  0001 C CNN
 	1    3200 2400
 	1    0    0    -1
 $EndComp
 $Comp
-L R R?
+L R R9
 U 1 1 53918101
 P 2600 2550
-F 0 "R?" V 2680 2550 50  0000 C CNN
+F 0 "R9" V 2680 2550 50  0000 C CNN
 F 1 "180" V 2600 2550 50  0000 C CNN
+F 2 "" H 2600 2550 60  0001 C CNN
+F 3 "" H 2600 2550 60  0001 C CNN
 	1    2600 2550
 	-1   0    0    1
@@
 SENSOR 1
 $Comp
-L TCRT1000 U?
+L TCRT1000 U3
 U 1 1 53918114
 P 3200 3250
-F 0 "U?" H 3200 3250 60  0000 C CNN
+F 0 "U3" H 3200 3250 60  0000 C CNN
 F 1 "TCRT1000" H 3450 3450 60  0000 C CNN
 F 2 "TCRT1000" H 2950 3450 60  0000 C CNN
+F 3 "" H 3200 3250 60  0001 C CNN
 	1    3200 3250
 	1    0    0    -1
 $EndComp
 $Comp
-L R R?
+L R R10
 U 1 1 5391811A
 P 2600 3400
-F 0 "R?" V 2680 3400 50  0000 C CNN
+F 0 "R10" V 2680 3400 50  0000 C CNN
 F 1 "180" V 2600 3400 50  0000 C CNN
+F 2 "" H 2600 3400 60  0001 C CNN
+F 3 "" H 2600 3400 60  0001 C CNN
 	1    2600 3400
 	-1   0    0    1
@@
 SENSOR 3
 $Comp
-L TCRT1000 U?
+L TCRT1000 U5
 U 1 1 5391812D
 P 4850 2400
-F 0 "U?" H 4850 2400 60  0000 C CNN
+F 0 "U5" H 4850 2400 60  0000 C CNN
 F 1 "TCRT1000" H 5100 2600 60  0000 C CNN
 F 2 "TCRT1000" H 4600 2600 60  0000 C CNN
+F 3 "" H 4850 2400 60  0001 C CNN
 	1    4850 2400
 	1    0    0    -1
 $EndComp
 $Comp
-L R R?
+L R R12
 U 1 1 53918133
 P 4250 2550
-F 0 "R?" V 4330 2550 50  0000 C CNN
+F 0 "R12" V 4330 2550 50  0000 C CNN
 F 1 "180" V 4250 2550 50  0000 C CNN
+F 2 "" H 4250 2550 60  0001 C CNN
+F 3 "" H 4250 2550 60  0001 C CNN
 	1    4250 2550
 	-1   0    0    1
@@
 SENSOR 2
 $Comp
-L TCRT1000 U?
+L TCRT1000 U6
 U 1 1 53918146
 P 4850 3250
-F 0 "U?" H 4850 3250 60  0000 C CNN
+F 0 "U6" H 4850 3250 60  0000 C CNN
 F 1 "TCRT1000" H 5100 3450 60  0000 C CNN
 F 2 "TCRT1000" H 4600 3450 60  0000 C CNN
+F 3 "" H 4850 3250 60  0001 C CNN
 	1    4850 3250
 	1    0    0    -1
 $EndComp
 $Comp
-L R R?
+L R R13
 U 1 1 5391814C
 P 4250 3400
-F 0 "R?" V 4330 3400 50  0000 C CNN
+F 0 "R13" V 4330 3400 50  0000 C CNN
 F 1 "180" V 4250 3400 50  0000 C CNN
+F 2 "" H 4250 3400 60  0001 C CNN
+F 3 "" H 4250 3400 60  0001 C CNN
 	1    4250 3400
 	-1   0    0    1
@@
 SENSOR 4
 $Comp
-L TCRT1000 SERVO_U?
+L TCRT1000 U4
 U 1 1 5391815F
 P 3200 4100
-F 0 "SERVO_U?" H 3200 4100 60  0000 C CNN
+F 0 "U4" H 3200 4100 60  0000 C CNN
 F 1 "TCRT1000" H 3450 4300 60  0000 C CNN
 F 2 "TCRT1000" H 2950 4300 60  0000 C CNN
+F 3 "" H 3200 4100 60  0001 C CNN
 	1    3200 4100
 	1    0    0    -1
 $EndComp
 $Comp
-L R R?
+L R R11
 U 1 1 53918165
 P 2600 4250
-F 0 "R?" V 2680 4250 50  0000 C CNN
+F 0 "R11" V 2680 4250 50  0000 C CNN
 F 1 "180" V 2600 4250 50  0000 C CNN
+F 2 "" H 2600 4250 60  0001 C CNN
+F 3 "" H 2600 4250 60  0001 C CNN
 	1    2600 4250
 	-1   0    0    1
@@
 SENSOR 5
 $Comp
-L TCRT1000 SERVO_U?
+L TCRT1000 U7
 U 1 1 53918178
 P 4850 4100
-F 0 "SERVO_U?" H 4850 4100 60  0000 C CNN
+F 0 "U7" H 4850 4100 60  0000 C CNN
 F 1 "TCRT1000" H 5100 4300 60  0000 C CNN
 F 2 "TCRT1000" H 4600 4300 60  0000 C CNN
+F 3 "" H 4850 4100 60  0001 C CNN
 	1    4850 4100
 	1    0    0    -1
 $EndComp
 $Comp
-L R R?
+L R R14
 U 1 1 5391817E
 P 4250 4250
-F 0 "R?" V 4330 4250 50  0000 C CNN
+F 0 "R14" V 4330 4250 50  0000 C CNN
 F 1 "180" V 4250 4250 50  0000 C CNN
+F 2 "" H 4250 4250 60  0001 C CNN
+F 3 "" H 4250 4250 60  0001 C CNN
 	1    4250 4250
 	-1   0    0    1

Commit message: Reempezado el pcb.
Changed lines of the file:
@@
 Sheet 3 4
 Title ""
-Date "14 jun 2014"
+Date "5 jul 2014"
 Rev ""
 Comp ""
@@
 	-1   0    0    1
 $EndComp
-Text Label 3800 3750 2    60   ~ 0
+Text Label 3800 4600 2    60   ~ 0
 SENSOR 3
 $Comp
@@
 	-1   0    0    1
 $EndComp
-Text Label 5450 2900 2    60   ~ 0
+Text Label 3800 3750 2    60   ~ 0
 SENSOR 2
 $Comp
@@
 	-1   0    0    1
 $EndComp
-Text Label 5450 3750 2    60   ~ 0
+Text Label 5450 2900 2    60   ~ 0
 SENSOR 4
 $Comp
@@
 	-1   0    0    1
 $EndComp
-Text Label 3800 4600 2    60   ~ 0
+Text Label 5450 3750 2    60   ~ 0
 SENSOR 5
 $Comp

Commit message: Colocados 8 sensores en la placa.
Parts:
- added R12, R16: 180, symbol R
- added R23, R24: 100, symbol R
- added RV7, RV8: POT 20 k, symbol POT
- added U5, U9: TCRT1000, TCRT1000, symbol TCRT1000
- renumbered R12 to R13, R13 to R14, R14 to R15, R15 to R17, R16 to R18, R17 to R19, R18 to R20, R19 to R21, R20 to R22, U5 to U6, U6 to U7, U7 to U8
Connections:
- net labels added: SENSOR 7, SENSOR 8, Sensor 7, Sensor 8
- wire segments 94 -> 122
Other:
- moved on the sheet: R17, R18, R19, R20, R21, R22, RV1, RV2, RV3, RV4, RV5, RV6
